File: RASBB/Hardware/Rev.B/Design/RASBB.kicad_sch (KiCad schematic)
At the start: 42 parts

Commit message: Rev B
Config Flash 2 modified, Termination added to LVDS lines
Parts:
- added R168, R169, R170, R171, R172, R173, R174, R175, R176, R177, R178, R179, R180, R181, R182, R183, R184: 100, Resistor_SMD:R_0201_0603Metric, symbol Device:R_Small
Connections:
- net FPGA-01/F1_B35_A1: now also R175.1
- net FPGA-01/F1_B35_A3: now also R179.1
- net FPGA-01/F1_B35_A4: now also R179.2
- net FPGA-01/F1_B35_A5: now also R181.1
- net FPGA-01/F1_B35_A6: now also R181.2
- net FPGA-01/F1_B35_B1: now also R175.2
- net FPGA-01/F1_B35_B2: now also R177.1
- net FPGA-01/F1_B35_B3: now also R177.2
- net FPGA-01/F1_B35_B4: now also R182.1
- net FPGA-01/F1_B35_B6: now also R183.1
- net FPGA-01/F1_B35_B7: now also R183.2
- net FPGA-01/F1_B35_C1: now also R178.1
- net FPGA-01/F1_B35_C2: now also R178.2
- net FPGA-01/F1_B35_C4: now also R182.2
- net FPGA-01/F1_B35_C5: now also R184.1
- net FPGA-01/F1_B35_C6: now also R184.2
- net FPGA-01/F1_B35_D4: now also R180.1
- net FPGA-01/F1_B35_D5: now also R180.2
- net FPGA-01/F1_B35_E1: now also R173.1
- net FPGA-01/F1_B35_E5: now also R176.1
- net FPGA-01/F1_B35_E6: now also R176.2
- net FPGA-01/F1_B35_F1: now also R173.2
- net FPGA-01/F1_B35_F3: now also R174.1
- net FPGA-01/F1_B35_F4: now also R174.2
- net FPGA-01/F1_B35_G1: now also R171.1
- net FPGA-01/F1_B35_G2: now also R172.1
- net FPGA-01/F1_B35_G3: now also R170.1
- net FPGA-01/F1_B35_G4: now also R170.2
- net FPGA-01/F1_B35_H1: now also R171.2
- net FPGA-01/F1_B35_H2: now also R172.2
- net FPGA-01/F1_B35_J2: now also R168.1
- net FPGA-01/F1_B35_J3: now also R168.2
- net FPGA-01/F1_B35_K1: now also R169.1
- net FPGA-01/F1_B35_K2: now also R169.2
