File: RASANT2400/Hardware/KiCad/RASANT2400.kicad_sch (KiCad schematic)
At the start: 0 parts

Commit message: added license note on silkscreen removed older RASBB revision
Other:
- title: (none) -> 2.4GHz 3 Element Yagi Antenna 
Changed lines of the file:
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@@
 	(generator_version "10.0")
 	(paper "A4")
+	(title_block
+		(title "2.4GHz 3 Element Yagi Antenna ")
+		(date "2026-05-30")
+		(rev "1.0")
+	)
 	(sheet_instances
 		(path "/"
