File: RASBB/Hardware/Rev.C/Design/RASBB.kicad_pcb (KiCad board)
At the start: 8 copper layers, 167.2 x 95.4 mm, 707 parts, among them IC1 RT6365GSP, IC10 MT41K128M16JT-107:K, IC11 TPD12S016PWR, IC12 STM32H743VGT6, IC13 SX1280IMLTRT, IC14 LAN8742AI-CZ-TR, IC15 DS90LV028AQDQFRQ1, IC2 TPS56528DDAR, IC3 TPS563201DDCR, IC4 TPS56528DDAR, IC5 S25FL128LAGMFI010, IC6 TS3A5018DBQR, IC7 S25FL128LAGMFI010, IC8 TS3A5018DBQR, IC9 MT41K128M16JT-107:K, J1 PJ-002AH-SMT-TR, J10 ZX-PZ1.27-2-5PWZ, J11 Conn_Coaxial, J12 AudioJack4, J13 Conn_01x06_Socket, J14 636101112001, J15 Conn_01x06_Socket, J16 Conn_01x02_Pin, J17 Conn_01x02_Pin, J18 Conn_01x02_Pin, J19 HC-WK88-H16-DB, J2 HR911196AE, J20 Conn_01x02_Pin, J3 HDMI-001A, J4 X3157WS-98-9TV30, J5 FH12-50S-0.5SV, J7 USB_C_Receptacle, J8 ZX-PZ1.27-2-5PWZ, J9 KF2EDGR-3.5-2P, Q1 DMN6075S, SW1 435451019820, SW2 435451019820, T1 15FB-30NL, U1 SZMMSZ4702T1G, U10 XC7A100T-CSG324, U11 XC7A100T-CSG324, U12 RTL8211E-VB-CG, U2 SI2324DS-T1-GE3, U3 SIC453ED-T1-GE3, U4 JW5026, U5 TLV9001DBVR, U6 CH340E, U7 AHT20, U8 LM386, U9 LM321, X1 OT2EL4C4JI-111OLP-50M, X3 OT2EL4C4JI-111OLP-50M, X4 OT2EL4C4JI-111OLP-50M, Y1 X503220MSB2GI, Y2 XC21M4-52.000-F10NNHPL, Y3 25MHz

Commit message: RevC_06
Parts:
- removed D17, D18, D19: A-SP192DGHC-C01-4T, LED_SMD:LED_0603_1608Metric
- removed R128, R129, R130: 715, Resistor_SMD:R_0402_1005Metric
- removed R208, R209: 0, Resistor_SMD:R_1206_3216Metric
- added C324: 100nF, Capacitor_SMD:C_0402_1005Metric, F.Cu at (189.8, 98.0)
- added J6: Conn_01x03, Connector_PinHeader_2.54mm:PinHeader_1x03_P2.54mm_Vertical, F.Cu at (112.0, 115.5)
- added R211: 0.005, Resistor_SMD:R_2512_6332Metric, F.Cu at (188.7, 40.6)
- added R212: 270, Resistor_SMD:R_0402_1005Metric, B.Cu at (263.6, 40.9)
- added R213: 270, Resistor_SMD:R_0402_1005Metric, B.Cu at (266.6, 40.9)
- added R214: 270, Resistor_SMD:R_0402_1005Metric, B.Cu at (257.3, 46.6)
- added R215: 270, Resistor_SMD:R_0402_1005Metric, B.Cu at (255.2, 44.5)
- added R216: 270, Resistor_SMD:R_0402_1005Metric, B.Cu at (236.2, 37.7)
- added R217: 270, Resistor_SMD:R_0402_1005Metric, B.Cu at (239.2, 37.7)
- added R218: 270, Resistor_SMD:R_0402_1005Metric, B.Cu at (247.8, 46.6)
- added R219: 270, Resistor_SMD:R_0402_1005Metric, B.Cu at (249.9, 44.6)
- added R220: 0.005, Resistor_SMD:R_2512_6332Metric, F.Cu at (216.7, 45.9)
- added R221: 0.005, Resistor_SMD:R_2512_6332Metric, F.Cu at (216.4, 64.9)
- added R222: 0.005, Resistor_SMD:R_2512_6332Metric, F.Cu at (197.3, 50.5)
- added R223: 0.005, Resistor_SMD:R_2512_6332Metric, F.Cu at (143.7, 40.5)
- C183, C322, C74: value tbd -> 1nF
- C4: value 10uF/100V -> 10uF, 100V
- J1: value PJ-002AH-SMT-TR -> DC_12V_IN
- J10: value ZX-PZ1.27-2-5PWZ -> STM32_JTAG
- J11: value Conn_Coaxial -> LORA_ANT
- J12: value AudioJack4 -> AUDIO
- J13: value Conn_01x06_Socket -> FPGA1_JTAG
- J14: value 636101112001 -> SYNC_40MHZ
- J15: value Conn_01x06_Socket -> FPGA2_JTAG
- J16: value Conn_01x02_Pin -> FPGA1_CLK_OUT
- J17: value Conn_01x02_Pin -> FE_3V3_MEAS
- J18: value Conn_01x02_Pin -> FPGA2_CLK_OUT
- J19: value HC-WK88-H16-DB -> ETH_100M_POE
- J2: value HR911196AE -> ETH_1G
- J20: value Conn_01x02_Pin -> PWM_DAC_OUT
- J3: value HDMI-001A -> HDMI
- J4: value X3157WS-98-9TV30 -> FRONTEND
- J5: value FH12-50S-0.5SV -> ICON
- J7: value USB_C_Receptacle -> USB_UART
- J8: value ZX-PZ1.27-2-5PWZ -> STM32_DEBUG
- J9: value KF2EDGR-3.5-2P -> ALARM_OUT
- R10, R101, R107, R114, R115, R116, R117, R118, R119, R120, R57, R58, R59, R60, R61, R62, R74, R76, R9: value 4.7K -> 4K7
- R26, U1: moved to F.Cu
- moved C320 23.2 mm to (264.6, 40.9), turned to 90 degrees
- moved C321 23.2 mm to (265.6, 40.9), turned to 90 degrees
- moved C309 12.1 mm to (238.2, 37.7)
- moved C288 12.0 mm to (237.2, 37.7)
- moved R114 11.2 mm to (188.5, 98.0), turned to 90 degrees
- moved R116 10.8 mm to (185.1, 98.4), turned to 180 degrees
- moved R115 10.6 mm to (183.2, 100.0)
- moved C240 9.93 mm to (256.6, 45.9), turned to 45 degrees
- moved D20 9.83 mm to (113.8, 42.2), turned to 90 degrees
- moved D21 9.18 mm to (118.8, 42.2), turned to 90 degrees
- moved C286 8.45 mm to (255.9, 45.2), turned to 45 degrees
- moved U1 8.28 mm to (215.4, 57.1), turned to -90 degrees
- moved R131 7.23 mm to (115.2, 41.8), turned to 90 degrees
- moved R26 5.16 mm to (217.8, 57.0), turned to 90 degrees
- moved R138 4.93 mm to (120.2, 41.8), turned to 90 degrees
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Connections:
- net +1V0 renamed /FPGA-01/1V0
- net +1V35 renamed /DDR3-01/VCCO_DDR3
- net +1V8 renamed /FPGA-01/1V8
- net +5V renamed /Audio_IN-OUT/5V0
- net /Config-SPI FLASH/SCK_Flash_FPGA2 renamed /Config-SPI FLASH/SCK_FLASH_FPGA2
- net /Config-SPI FLASH/SI_Flash_FPGA2 renamed /Config-SPI FLASH/SI_FLASH_FPGA2
- net /Config-SPI FLASH/SO_Flash_FPGA2 renamed /Config-SPI FLASH/SO_FLASH_FPGA2
- net /Inteconnect/Debug_A0 renamed /Interconnect/Debug_A0
- net /Inteconnect/Debug_A1 renamed /Interconnect/Debug_A1
- net /Inteconnect/Debug_A2 renamed /Interconnect/Debug_A2
- net /Inteconnect/Debug_A3 renamed /Interconnect/Debug_A3
- net /Inteconnect/Debug_A4 renamed /Interconnect/Debug_A4
- net /Inteconnect/Debug_A5 renamed /Interconnect/Debug_A5
- net /Inteconnect/Debug_A6 renamed /Interconnect/Debug_A6
- net /Inteconnect/Debug_A7 renamed /Interconnect/Debug_A7
- net /Inteconnect/Debug_D0 renamed /Interconnect/Debug_D0
- net /Inteconnect/Debug_D1 renamed /Interconnect/Debug_D1
- net /Inteconnect/Debug_D10 renamed /Interconnect/Debug_D10
- net /Inteconnect/Debug_D11 renamed /Interconnect/Debug_D11
- net /Inteconnect/Debug_D12 renamed /Interconnect/Debug_D12
- net /Inteconnect/Debug_D13 renamed /Interconnect/Debug_D13
- net /Inteconnect/Debug_D14 renamed /Interconnect/Debug_D14
- net /Inteconnect/Debug_D15 renamed /Interconnect/Debug_D15
- net /Inteconnect/Debug_D16 renamed /Interconnect/Debug_D16
- net /Inteconnect/Debug_D17 renamed /Interconnect/Debug_D17
- net /Inteconnect/Debug_D18 renamed /Interconnect/Debug_D18
- net /Inteconnect/Debug_D19 renamed /Interconnect/Debug_D19
- net /Inteconnect/Debug_D2 renamed /Interconnect/Debug_D2
- net /Inteconnect/Debug_D20 renamed /Interconnect/Debug_D20
- net /Inteconnect/Debug_D21 renamed /Interconnect/Debug_D21
- net /Inteconnect/Debug_D22 renamed /Interconnect/Debug_D22
- net /Inteconnect/Debug_D23 renamed /Interconnect/Debug_D23
- net /Inteconnect/Debug_D24 renamed /Interconnect/Debug_D24
- net /Inteconnect/Debug_D25 renamed /Interconnect/Debug_D25
- net /Inteconnect/Debug_D26 renamed /Interconnect/Debug_D26
- net /Inteconnect/Debug_D27 renamed /Interconnect/Debug_D27
- net /Inteconnect/Debug_D28 renamed /Interconnect/Debug_D28
- net /Inteconnect/Debug_D29 renamed /Interconnect/Debug_D29
- net /Inteconnect/Debug_D3 renamed /Interconnect/Debug_D3
- net /Inteconnect/Debug_D30 renamed /Interconnect/Debug_D30
- net /Inteconnect/Debug_D31 renamed /Interconnect/Debug_D31
- net /Inteconnect/Debug_D4 renamed /Interconnect/Debug_D4
- net /Inteconnect/Debug_D5 renamed /Interconnect/Debug_D5
- net /Inteconnect/Debug_D6 renamed /Interconnect/Debug_D6
- net /Inteconnect/Debug_D7 renamed /Interconnect/Debug_D7
- net /Inteconnect/Debug_D8 renamed /Interconnect/Debug_D8
- net /Inteconnect/Debug_D9 renamed /Interconnect/Debug_D9
- C123 pad 1: +3V3 -> /Audio_IN-OUT/3V3
- C125 pad 2: +3V3 -> /Audio_IN-OUT/3V3
- C126 pad 1: +3V3 -> /Audio_IN-OUT/3V3
- C127 pad 1: +3V3 -> /Audio_IN-OUT/3V3
- C128 pad 1: +3V3 -> /Audio_IN-OUT/3V3
- C129 pad 1: +3V3 -> /Audio_IN-OUT/3V3
- C131 pad 1: +3V3 -> /Audio_IN-OUT/3V3
- C133 pad 1: +3V3 -> /Audio_IN-OUT/3V3
- C134 pad 1: +3V3 -> /Audio_IN-OUT/3V3
- C135 pad 1: +3V3 -> /Audio_IN-OUT/3V3
- C136 pad 1: +3V3 -> /Audio_IN-OUT/3V3
- C137 pad 1: +3V3 -> /Audio_IN-OUT/3V3
- C138 pad 1: +3V3 -> /Audio_IN-OUT/3V3
- C164 pad 1: +3V3 -> /Audio_IN-OUT/3V3
- C17 pad 1: +12V -> Net-(U3B-PVIN)
- C170 pad 1: +3V3 -> /Audio_IN-OUT/3V3
- C172 pad 1: +3V3 -> /Audio_IN-OUT/3V3
- C173 pad 1: +3V3 -> /Audio_IN-OUT/3V3
- C18 pad 1: +12V -> Net-(U3B-PVIN)
- C188 pad 2: +3V3 -> /Audio_IN-OUT/3V3
- C195 pad 1: +3V3 -> /Audio_IN-OUT/3V3
- C199 pad 1: +3V3 -> /Audio_IN-OUT/3V3
- C202 pad 2: +3V3 -> /Audio_IN-OUT/3V3
- C204 pad 2: +3V3 -> /Audio_IN-OUT/3V3
- C21 pad 1: +12V -> Net-(IC2-VIN)
- C22 pad 1: +12V -> Net-(IC4-VIN)
- C221 pad 1: +3V3 -> /Audio_IN-OUT/3V3
- C222 pad 1: +3V3 -> /Audio_IN-OUT/3V3
- C23 pad 1: +12V -> Net-(IC3-VIN)
- C233 pad 1: +3V3 -> /Audio_IN-OUT/3V3
- C234 pad 1: +3V3 -> /Audio_IN-OUT/3V3
- C235 pad 1: +3V3 -> /Audio_IN-OUT/3V3
- C236 pad 1: +3V3 -> /Audio_IN-OUT/3V3
- C237 pad 1: +3V3 -> /Audio_IN-OUT/3V3
- C239 pad 1: +3V3 -> /Audio_IN-OUT/3V3
- C24 pad 1: +12V -> Net-(IC2-VIN)
- C240 pad 1: /FPGA-01/F1_B15_B18 -> /HDMI/HDMI_D1_P
- C240 pad 2: /HDMI/HDMI_D2_P -> /HDMI/TMDS_D1_P
- C241 pad 1: +3V3 -> /Audio_IN-OUT/3V3
- C242 pad 1: +3V3 -> /Audio_IN-OUT/3V3
- C243 pad 1: +3V3 -> /Audio_IN-OUT/3V3
- C244 pad 1: +3V3 -> /Audio_IN-OUT/3V3
- C245 pad 1: +3V3 -> /Audio_IN-OUT/3V3
- C246 pad 1: +3V3 -> /Audio_IN-OUT/3V3
- C247 pad 1: +3V3 -> /Audio_IN-OUT/3V3
- C248 pad 1: +3V3 -> /Audio_IN-OUT/3V3
- C249 pad 1: +3V3 -> /Audio_IN-OUT/3V3
- C25 pad 1: +12V -> Net-(IC4-VIN)
- C250 pad 1: +3V3 -> /Audio_IN-OUT/3V3
- C251 pad 1: +3V3 -> /Audio_IN-OUT/3V3
- C252 pad 1: +3V3 -> /Audio_IN-OUT/3V3
- C253 pad 1: +3V3 -> /Audio_IN-OUT/3V3
- C254 pad 1: +3V3 -> /Audio_IN-OUT/3V3
- C255 pad 1: +3V3 -> /Audio_IN-OUT/3V3
- C256 pad 2: +3V3 -> /Audio_IN-OUT/3V3
- C257 pad 1: +3V3 -> /Audio_IN-OUT/3V3
- C26 pad 1: +12V -> Net-(IC3-VIN)
- C27 pad 1: +12V -> Net-(IC2-VIN)
- C270 pad 1: +3V3 -> /Audio_IN-OUT/3V3
- C28 pad 1: +12V -> Net-(IC4-VIN)
- C286 pad 1: /FPGA-01/F1_B15_A18 -> /HDMI/HDMI_D1_N
- C286 pad 2: /HDMI/HDMI_D2_N -> /HDMI/TMDS_D1_N
- C288 pad 1: /FPGA-01/F1_B15_A15 -> /HDMI/HDMI_D0_P
- C288 pad 2: /HDMI/HDMI_D1_P -> /HDMI/TMDS_D0_P
- C29 pad 1: +12V -> Net-(U4-VIN)
- C305 pad 1: +3V3 -> /Audio_IN-OUT/3V3
- C306 pad 1: +3V3 -> /Audio_IN-OUT/3V3
- C309 pad 1: /FPGA-01/F1_B15_A16 -> /HDMI/HDMI_D0_N
- C309 pad 2: /HDMI/HDMI_D1_N -> /HDMI/TMDS_D0_N
- C31 pad 1: +12V -> Net-(IC3-VIN)
- C318 pad 1: /FPGA-01/F1_B15_B16 -> /HDMI/HDMI_CLK_P
- C318 pad 2: /HDMI/HDMI_D0_P -> /HDMI/TMDS_CK_P
- C319 pad 1: /FPGA-01/F1_B15_B17 -> /HDMI/HDMI_CLK_N
- C319 pad 2: /HDMI/HDMI_D0_N -> /HDMI/TMDS_CK_N
- C320 pad 1: /FPGA-01/F1_B15_A13 -> /HDMI/HDMI_D2_P
- C320 pad 2: /HDMI/HDMI_CLK_P -> /HDMI/TMDS_D2_P
- C321 pad 1: /FPGA-01/F1_B15_A14 -> /HDMI/HDMI_D2_N
- C321 pad 2: /HDMI/HDMI_CLK_N -> /HDMI/TMDS_D2_N
- C323 pad 1: +3V3 -> /Audio_IN-OUT/3V3
- C326 pad 1: +3V3 -> /Audio_IN-OUT/3V3
- C327 pad 1: +3V3 -> /Audio_IN-OUT/3V3
- C328 pad 1: +3V3 -> /Audio_IN-OUT/3V3
- C329 pad 1: +3V3 -> /Audio_IN-OUT/3V3
- C330 pad 1: +3V3 -> /Audio_IN-OUT/3V3
- C331 pad 1: +3V3 -> /Audio_IN-OUT/3V3
- C332 pad 1: +3V3 -> /Audio_IN-OUT/3V3
- C333 pad 1: +3V3 -> /Audio_IN-OUT/3V3
- C334 pad 1: +3V3 -> /Audio_IN-OUT/3V3
- C335 pad 1: +3V3 -> /Audio_IN-OUT/3V3
- C336 pad 1: +3V3 -> /Audio_IN-OUT/3V3
- C337 pad 1: +3V3 -> /Audio_IN-OUT/3V3
- C338 pad 1: +3V3 -> /Audio_IN-OUT/3V3
- C339 pad 1: +3V3 -> /Audio_IN-OUT/3V3
- C346 pad 1: +3V3 -> /Audio_IN-OUT/3V3
- C347 pad 1: +3V3 -> /Audio_IN-OUT/3V3
- C348 pad 1: +3V3 -> /Audio_IN-OUT/3V3
- C349 pad 1: +3V3 -> /Audio_IN-OUT/3V3
- C350 pad 1: +3V3 -> /Audio_IN-OUT/3V3
- C351 pad 1: +3V3 -> /Audio_IN-OUT/3V3
- C352 pad 1: +3V3 -> /Audio_IN-OUT/3V3
- C354 pad 1: +12V -> Net-(U3B-PVIN)
- C355 pad 1: +12V -> Net-(U3B-PVIN)
- C356 pad 1: +12V -> Net-(U3B-PVIN)
- C363 pad 1: +3V3 -> /Audio_IN-OUT/3V3
- C364 pad 1: +3V3 -> /Audio_IN-OUT/3V3
- C43 pad 1: +3V3 -> /Audio_IN-OUT/3V3
- C51 pad 1: +3V3 -> /Audio_IN-OUT/3V3
- C53 pad 2: +3V3 -> /Audio_IN-OUT/3V3
- C56 pad 2: +3V3 -> /Audio_IN-OUT/3V3
- C58 pad 1: +3V3 -> /Audio_IN-OUT/3V3
- C59 pad 1: +3V3 -> /Audio_IN-OUT/3V3
- C60 pad 1: +3V3 -> /Audio_IN-OUT/3V3
- C61 pad 1: +3V3 -> /Audio_IN-OUT/3V3
- C62 pad 1: +3V3 -> /Audio_IN-OUT/3V3
- C64 pad 1: +3V3 -> /Audio_IN-OUT/3V3
- C68 pad 1: +3V3 -> /Audio_IN-OUT/3V3
- C70 pad 1: +3V3 -> /Audio_IN-OUT/3V3
- C71 pad 1: +3V3 -> /Audio_IN-OUT/3V3
- C72 pad 1: +3V3 -> /Audio_IN-OUT/3V3
- D10 pad 5: +3V3 -> /Audio_IN-OUT/3V3
- F2 pad 1: Net-(F2-Pad1) -> /PCIE/12V
- FB1 pad 1: +3V3 -> /Audio_IN-OUT/3V3
- FB2 pad 1: +3V3 -> /Audio_IN-OUT/3V3
- FB3 pad 1: +3V3 -> /Audio_IN-OUT/3V3
- IC11 pad 12: +3V3 -> /Audio_IN-OUT/3V3
- IC11 pad 24: +3V3 -> /Audio_IN-OUT/3V3
- IC11 pad 5: +3V3 -> /Audio_IN-OUT/3V3
- IC12 pad 100: +3V3 -> /Audio_IN-OUT/3V3
- IC12 pad 11: +3V3 -> /Audio_IN-OUT/3V3
- IC12 pad 27: +3V3 -> /Audio_IN-OUT/3V3
- IC12 pad 50: +3V3 -> /Audio_IN-OUT/3V3
- IC12 pad 6: +3V3 -> /Audio_IN-OUT/3V3
- IC12 pad 75: +3V3 -> /Audio_IN-OUT/3V3
- IC14 pad 9: +3V3 -> /Audio_IN-OUT/3V3
- IC15 pad 8: +3V3 -> /Audio_IN-OUT/3V3
- IC2 pad 8: +12V -> Net-(IC2-VIN)
- IC3 pad 3: +12V -> Net-(IC3-VIN)
- IC4 pad 8: +12V -> Net-(IC4-VIN)
- IC5 pad 8: +3V3 -> /Audio_IN-OUT/3V3
- IC6 pad 16: +3V3 -> /Audio_IN-OUT/3V3
- IC7 pad 8: +3V3 -> /Audio_IN-OUT/3V3
- IC8 pad 16: +3V3 -> /Audio_IN-OUT/3V3
- J10 pad 1: +3V3 -> /Audio_IN-OUT/3V3
- J10 pad 10: GND -> /uController/uC_NRST
- J10 pad 2: +3V3 -> /uController/DBG_JTMS_SWDIO
- J10 pad 3: /uController/uC_NRST -> GND
- J10 pad 4: unconnected-(J10-Pad4) -> /uController/DBG_JTCK_SWCLK
- J10 pad 5: /uController/DBG_JTDI -> GND
- J10 pad 7: /uController/DBG_JTMS_SWDIO -> unconnected-(J10-Pad7)
- J10 pad 8: /uController/DBG_JTCK_SWCLK -> /uController/DBG_JTDI
- J10 pad 9: /uController/DBG_JTCK_SWCLK -> GND
- J13 pad 6: +3V3 -> /Audio_IN-OUT/3V3
- J15 pad 6: +3V3 -> /Audio_IN-OUT/3V3
- J17 pad 1: +3V3 -> /Audio_IN-OUT/3V3
- J3 pad 1: /HDMI/HDMI_D2_P -> /HDMI/TMDS_D2_P
- J3 pad 10: /HDMI/HDMI_CLK_P -> /HDMI/TMDS_CK_P
- J3 pad 12: /HDMI/HDMI_CLK_N -> /HDMI/TMDS_CK_N
- J3 pad 3: /HDMI/HDMI_D2_N -> /HDMI/TMDS_D2_N
- J3 pad 4: /HDMI/HDMI_D1_P -> /HDMI/TMDS_D1_P
- J3 pad 6: /HDMI/HDMI_D1_N -> /HDMI/TMDS_D1_N
- J3 pad 7: /HDMI/HDMI_D0_P -> /HDMI/TMDS_D0_P
- J3 pad 9: /HDMI/HDMI_D0_N -> /HDMI/TMDS_D0_N
- J4 pad A32: unconnected-(J4-PadA32) -> GND
- J4 pad A33: unconnected-(J4-PadA33) -> GND
- J4 pad A34: unconnected-(J4-PadA34) -> GND
- J4 pad B01: Net-(J4-PadA01) -> Net-(J6-Pin_2)
- J4 pad B02: Net-(J4-PadA01) -> Net-(J6-Pin_2)
- J4 pad B03: Net-(J4-PadA01) -> Net-(J6-Pin_2)
- J4 pad B10: unconnected-(J4-PadB10) -> GND
- J4 pad B11: unconnected-(J4-PadB11) -> GND
- J4 pad B13: unconnected-(J4-PadB13) -> GND
- J4 pad B32: unconnected-(J4-PadB32) -> GND
- J5 pad 1: +3V3 -> /Audio_IN-OUT/3V3
- J5 pad 41: +3V3 -> /Audio_IN-OUT/3V3
- J8 pad 1: +3V3 -> /Audio_IN-OUT/3V3
- L11 pad 2: +3V3 -> /Audio_IN-OUT/3V3
- L6 pad 1: +3V3 -> /Audio_IN-OUT/3V3
- L8 pad 2: +3V3 -> /Audio_IN-OUT/3V3
- R10 pad 2: +3V3 -> /Audio_IN-OUT/3V3
- R103 pad 1: +3V3 -> /Audio_IN-OUT/3V3
- R107 pad 1: +3V3 -> /Audio_IN-OUT/3V3
- R114 pad 2: +3V3 -> /Audio_IN-OUT/3V3
- R115 pad 1: /uController/DBG_JTMS_SWDIO -> /uController/DBG_JTDO_SWO
- R115 pad 2: +3V3 -> /Audio_IN-OUT/3V3
- R116 pad 1: /uController/uC_NRST -> /uController/DBG_JTMS_SWDIO
- R116 pad 2: +3V3 -> /Audio_IN-OUT/3V3
- R117 pad 2: +3V3 -> /Audio_IN-OUT/3V3
- R118 pad 2: +3V3 -> /Audio_IN-OUT/3V3
- R119 pad 1: /uController/DBG_JTDO_SWO -> /uController/uC_NRST
- R119 pad 2: +3V3 -> /Audio_IN-OUT/3V3
- R125 pad 2: +3V3 -> /Audio_IN-OUT/3V3
- R127 pad 1: +3V3 -> /Audio_IN-OUT/3V3
- R131 pad 1: +3V3 -> /Audio_IN-OUT/3V3
- R132 pad 2: +3V3 -> /Audio_IN-OUT/3V3
- R133 pad 2: +3V3 -> /Audio_IN-OUT/3V3
- R136 pad 2: +3V3 -> /Audio_IN-OUT/3V3
- R137 pad 2: +3V3 -> /Audio_IN-OUT/3V3
- R156 pad 1: +3V3 -> /Audio_IN-OUT/3V3
- R164 pad 1: +3V3 -> /Audio_IN-OUT/3V3
- R185 pad 2: +3V3 -> /Audio_IN-OUT/3V3
- R191 pad 1: +3V3 -> /Audio_IN-OUT/3V3
- R192 pad 1: +3V3 -> /Audio_IN-OUT/3V3
- R196 pad 1: +3V3 -> /Audio_IN-OUT/3V3
- R197 pad 1: +3V3 -> /Audio_IN-OUT/3V3
- R198 pad 1: +3V3 -> /Audio_IN-OUT/3V3
- R199 pad 1: +3V3 -> /Audio_IN-OUT/3V3
- R200 pad 2: +3V3 -> /Audio_IN-OUT/3V3
- R201 pad 2: +3V3 -> /Audio_IN-OUT/3V3
- R204 pad 1: +3V3 -> /Audio_IN-OUT/3V3
- R205 pad 1: +3V3 -> /Audio_IN-OUT/3V3
- R206 pad 1: +3V3 -> /Audio_IN-OUT/3V3
- R207 pad 1: +3V3 -> /Audio_IN-OUT/3V3
- R36 pad 2: +12V -> Net-(U3B-PVIN)
- R42 pad 1: +12V -> Net-(U4-VIN)
- R5 pad 1: +3V3 -> /Audio_IN-OUT/3V3
- R51 pad 2: +3V3 -> /Audio_IN-OUT/3V3
- R53 pad 1: +3V3 -> /Audio_IN-OUT/3V3
- R54 pad 1: +3V3 -> /Audio_IN-OUT/3V3
- R55 pad 1: +3V3 -> /Audio_IN-OUT/3V3
- R56 pad 1: +3V3 -> /Audio_IN-OUT/3V3
- R57 pad 2: +3V3 -> /Audio_IN-OUT/3V3
- R58 pad 2: +3V3 -> /Audio_IN-OUT/3V3
- R59 pad 1: +3V3 -> /Audio_IN-OUT/3V3
- R61 pad 2: +3V3 -> /Audio_IN-OUT/3V3
- R62 pad 2: +3V3 -> /Audio_IN-OUT/3V3
- R67 pad 2: +3V3 -> /Audio_IN-OUT/3V3
- R72 pad 2: +3V3 -> /Audio_IN-OUT/3V3
- R75 pad 1: +3V3 -> /Audio_IN-OUT/3V3
- R77 pad 1: +3V3 -> /Audio_IN-OUT/3V3
- R9 pad 2: +3V3 -> /Audio_IN-OUT/3V3
- R96 pad 1: +3V3 -> /Audio_IN-OUT/3V3
- TP1 pad 1: +3V3 -> /Audio_IN-OUT/3V3
- U10 pad A13: /FPGA-01/F1_B15_A13 -> /HDMI/HDMI_CLK_P
- U10 pad A14: /FPGA-01/F1_B15_A14 -> /HDMI/HDMI_CLK_N
- U10 pad A15: /FPGA-01/F1_B15_A15 -> /HDMI/HDMI_D1_P
- U10 pad A16: /FPGA-01/F1_B15_A16 -> /HDMI/HDMI_D1_N
- U10 pad A17: +3V3 -> /Audio_IN-OUT/3V3
- U10 pad A18: /FPGA-01/F1_B15_A18 -> /HDMI/HDMI_D2_N
- U10 pad B16: /FPGA-01/F1_B15_B16 -> /HDMI/HDMI_D0_P
- U10 pad B17: /FPGA-01/F1_B15_B17 -> /HDMI/HDMI_D0_N
- U10 pad B18: /FPGA-01/F1_B15_B18 -> /HDMI/HDMI_D2_P
- U10 pad C13: +3V3 -> /Audio_IN-OUT/3V3
- U10 pad D16: +3V3 -> /Audio_IN-OUT/3V3
- U10 pad G15: +3V3 -> /Audio_IN-OUT/3V3
- U10 pad H18: +3V3 -> /Audio_IN-OUT/3V3
- U10 pad K14: +3V3 -> /Audio_IN-OUT/3V3
- U10 pad L17: +3V3 -> /Audio_IN-OUT/3V3
- U10 pad N13: +3V3 -> /Audio_IN-OUT/3V3
- U10 pad P12: +3V3 -> /Audio_IN-OUT/3V3
- U10 pad P16: +3V3 -> /Audio_IN-OUT/3V3
- U10 pad P8: +3V3 -> /Audio_IN-OUT/3V3
- U10 pad R9: +3V3 -> /Audio_IN-OUT/3V3
- U10 pad T12: +3V3 -> /Audio_IN-OUT/3V3
- U10 pad U15: +3V3 -> /Audio_IN-OUT/3V3
- U10 pad V18: +3V3 -> /Audio_IN-OUT/3V3
- U11 pad A17: +3V3 -> /Audio_IN-OUT/3V3
- U11 pad A7: +3V3 -> /Audio_IN-OUT/3V3
- U11 pad C13: +3V3 -> /Audio_IN-OUT/3V3
- U11 pad C3: +3V3 -> /Audio_IN-OUT/3V3
- U11 pad D16: +3V3 -> /Audio_IN-OUT/3V3
- U11 pad D6: +3V3 -> /Audio_IN-OUT/3V3
- U11 pad F2: +3V3 -> /Audio_IN-OUT/3V3
- U11 pad G15: +3V3 -> /Audio_IN-OUT/3V3
- U11 pad G5: +3V3 -> /Audio_IN-OUT/3V3
- U11 pad H18: +3V3 -> /Audio_IN-OUT/3V3
- U11 pad J1: +3V3 -> /Audio_IN-OUT/3V3
- U11 pad K14: +3V3 -> /Audio_IN-OUT/3V3
- U11 pad L17: +3V3 -> /Audio_IN-OUT/3V3
- U11 pad N13: +3V3 -> /Audio_IN-OUT/3V3
- U11 pad P12: +3V3 -> /Audio_IN-OUT/3V3
- U11 pad P16: +3V3 -> /Audio_IN-OUT/3V3
- U11 pad P8: +3V3 -> /Audio_IN-OUT/3V3
- U11 pad R9: +3V3 -> /Audio_IN-OUT/3V3
- U11 pad T12: +3V3 -> /Audio_IN-OUT/3V3
- U11 pad U15: +3V3 -> /Audio_IN-OUT/3V3
- U11 pad V18: +3V3 -> /Audio_IN-OUT/3V3
- U12 pad 15: +3V3 -> /Audio_IN-OUT/3V3
- U12 pad 21: +3V3 -> /Audio_IN-OUT/3V3
- U12 pad 37: +3V3 -> /Audio_IN-OUT/3V3
- U12 pad 38: +3V3 -> /Audio_IN-OUT/3V3
- U12 pad 44: +3V3 -> /Audio_IN-OUT/3V3
- U12 pad 45: +3V3 -> /Audio_IN-OUT/3V3
- U2 pad 2: GND -> /VSS_POE
- U2 pad 3: /VSS_POE -> GND
- U3 pad 1-3/34: +12V -> Net-(U3B-PVIN)
- U3 pad 23: +12V -> Net-(U3B-PVIN)
- U4 pad 5: +12V -> Net-(U4-VIN)
- U5 pad 5: +3V3 -> /Audio_IN-OUT/3V3
- U6 pad 10: +3V3 -> /Audio_IN-OUT/3V3
- U6 pad 7: +3V3 -> /Audio_IN-OUT/3V3
- U9 pad 5: +3V3 -> /Audio_IN-OUT/3V3
- X1 pad 1: +3V3 -> /Audio_IN-OUT/3V3
- X1 pad 4: +3V3 -> /Audio_IN-OUT/3V3
Routing:
- net /Audio_IN-OUT/3V3: track 0.00 -> 341.5 mm, vias 0 -> 222
- net +3V3: track 333.7 -> 0.00 mm, vias 215 -> 0
- net /PCIE/12V: track 0.00 -> 319.8 mm, vias 0 -> 27
- net +12V: track 267.7 -> 0.00 mm, vias 59 -> 0
- net /FPGA-01/F1_B15_B16: track 119.3 -> 0.00 mm, vias 2 -> 0
- net /FPGA-01/F1_B15_B17: track 119.3 -> 0.00 mm, vias 2 -> 0
- net /FPGA-01/F1_B15_A14: track 119.1 -> 0.00 mm, vias 2 -> 0
- net /FPGA-01/F1_B15_A13: track 117.2 -> 0.00 mm, vias 2 -> 0
- net /FPGA-01/F1_B15_A18: track 109.4 -> 0.00 mm, vias 2 -> 0
- net /HDMI/HDMI_CLK_N: track 21.6 -> 129.1 mm, vias 0 -> 2
- net /FPGA-01/F1_B15_B18: track 107.3 -> 0.00 mm, vias 2 -> 0
- net /HDMI/HDMI_CLK_P: track 22.6 -> 129.4 mm, vias 0 -> 2
- net /HDMI/HDMI_D0_P: track 31.2 -> 132.3 mm, vias 0 -> 2
- net /HDMI/HDMI_D0_N: track 29.7 -> 130.3 mm, vias 0 -> 2
- net /HDMI/HDMI_D2_P: track 49.4 -> 148.1 mm, vias 0 -> 2
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- added copper zone on F.Cu, net /Audio_IN-OUT/3V3
- added copper zone on In1.Cu, net /Audio_IN-OUT/3V3
- added copper zone on In6.Cu, net /Audio_IN-OUT/3V3
- added copper zone on In1.Cu, net /PCIE/12V
- added copper zone on F.Cu, net Net-(IC2-VIN)
- added copper zone on B.Cu, net Net-(IC3-VIN)
- added copper zone on F.Cu, net Net-(IC3-VIN)
- added copper zone on F.Cu, net Net-(IC4-VIN)
- added copper zone on F.Cu, net Net-(U3B-PVIN)
- added copper zone on In1.Cu, net Net-(U3B-PVIN)
- added copper zone on F.Cu, net Net-(U4-VIN)
- added copper zone on In1.Cu, net Net-(U4-VIN)
- removed copper zone on B.Cu, net +12V
- removed copper zone on F.Cu, net +12V
- removed copper zone on In1.Cu, net +12V
- removed copper zone on F.Cu, net +3V3
- removed copper zone on In1.Cu, net +3V3
- removed copper zone on In6.Cu, net +3V3
Other:
- board text added: "12V"
- board text removed: "1V"
- board text removed: "1V35"
- board text removed: "1V8"
- board text removed: "DNP R208 IF R209 IS POPULATED"
- board text removed: "RASBB Rev.B"
