File: RASBB/Hardware/Rev.C/Design/RASBB.kicad_pcb (KiCad board)
At the start: 8 copper layers, 167.2 x 95.4 mm, 714 parts, among them IC1 RT6365GSP, IC10 MT41K128M16JT-107:K, IC11 TPD12S016PWR, IC12 STM32H743VGT6, IC13 SX1280IMLTRT, IC14 LAN8742AI-CZ-TR, IC15 DS90LV028AQDQFRQ1, IC2 TPS56528DDAR, IC3 TPS563201DDCR, IC4 TPS56528DDAR, IC5 S25FL128LAGMFI010, IC6 TS3A5018DBQR, IC7 S25FL128LAGMFI010, IC8 TS3A5018DBQR, IC9 MT41K128M16JT-107:K, J1 DC_12V_IN, J10 STM32_JTAG, J11 LORA_ANT, J12 AUDIO, J13 FPGA1_JTAG, J14 SYNC_40MHZ, J15 FPGA2_JTAG, J16 FPGA1_CLK_OUT, J17 FE_3V3_MEAS, J18 FPGA2_CLK_OUT, J19 ETH_100M_POE, J2 ETH_1G, J20 PWM_DAC_OUT, J3 HDMI, J4 FRONTEND, J5 ICON, J6 Conn_01x03, J7 USB_UART, J8 STM32_DEBUG, J9 ALARM_OUT, Q1 DMN6075S, SW1 435451019820, SW2 435451019820, T1 15FB-30NL, U1 SZMMSZ4702T1G, U10 XC7A100T-CSG324, U11 XC7A100T-CSG324, U12 RTL8211E-VB-CG, U2 SI2324DS-T1-GE3, U3 SIC453ED-T1-GE3, U4 JW5026, U5 TLV9001DBVR, U6 CH340E, U7 AHT20, U8 LM386, U9 LM321, X1 OT2EL4C4JI-111OLP-50M, X3 OT2EL4C4JI-111OLP-50M, X4 OT2EL4C4JI-111OLP-50M, Y1 X503220MSB2GI, Y2 XC21M4-52.000-F10NNHPL, Y3 25MHz

Commit message: REV.C production data
Connections:
- C185 pad 1: /FPGA-01/1V0 -> /POWER/VSEN_P
- C189 pad 1: /FPGA-01/1V0 -> /POWER/VSEN_P
- C190 pad 1: /FPGA-01/1V0 -> /POWER/VSEN_P
- C193 pad 1: /FPGA-01/1V0 -> /POWER/VSEN_P
- C194 pad 1: /FPGA-01/1V0 -> /POWER/VSEN_P
- C197 pad 1: /FPGA-01/1V0 -> /POWER/VSEN_P
- C198 pad 1: /FPGA-01/1V0 -> /POWER/VSEN_P
- C201 pad 1: /FPGA-01/1V0 -> /POWER/VSEN_P
- C205 pad 1: /FPGA-01/1V0 -> /POWER/VSEN_P
- C207 pad 1: /FPGA-01/1V0 -> /POWER/VSEN_P
- C209 pad 1: /FPGA-01/1V0 -> /POWER/VSEN_P
- C211 pad 1: /FPGA-01/1V0 -> /POWER/VSEN_P
- C212 pad 1: /FPGA-01/1V0 -> /POWER/VSEN_P
- C213 pad 1: /FPGA-01/1V0 -> /POWER/VSEN_P
- C214 pad 1: /FPGA-01/1V0 -> /POWER/VSEN_P
- C215 pad 1: /FPGA-01/1V0 -> /POWER/VSEN_P
- C216 pad 1: /FPGA-01/1V0 -> /POWER/VSEN_P
- C217 pad 1: /FPGA-01/1V0 -> /POWER/VSEN_P
- C218 pad 1: /FPGA-01/1V0 -> /POWER/VSEN_P
- C219 pad 1: /FPGA-01/1V0 -> /POWER/VSEN_P
- C220 pad 1: /FPGA-01/1V0 -> /POWER/VSEN_P
- C269 pad 1: /FPGA-01/1V0 -> /POWER/VSEN_P
- C273 pad 1: /FPGA-01/1V0 -> /POWER/VSEN_P
- C274 pad 1: /FPGA-01/1V0 -> /POWER/VSEN_P
- C277 pad 1: /FPGA-01/1V0 -> /POWER/VSEN_P
- C278 pad 1: /FPGA-01/1V0 -> /POWER/VSEN_P
- C281 pad 1: /FPGA-01/1V0 -> /POWER/VSEN_P
- C282 pad 1: /FPGA-01/1V0 -> /POWER/VSEN_P
- C285 pad 1: /FPGA-01/1V0 -> /POWER/VSEN_P
- C289 pad 1: /FPGA-01/1V0 -> /POWER/VSEN_P
- C291 pad 1: /FPGA-01/1V0 -> /POWER/VSEN_P
- C293 pad 1: /FPGA-01/1V0 -> /POWER/VSEN_P
- C295 pad 1: /FPGA-01/1V0 -> /POWER/VSEN_P
- C296 pad 1: /FPGA-01/1V0 -> /POWER/VSEN_P
- C297 pad 1: /FPGA-01/1V0 -> /POWER/VSEN_P
- C298 pad 1: /FPGA-01/1V0 -> /POWER/VSEN_P
- C299 pad 1: /FPGA-01/1V0 -> /POWER/VSEN_P
- C300 pad 1: /FPGA-01/1V0 -> /POWER/VSEN_P
- C301 pad 1: /FPGA-01/1V0 -> /POWER/VSEN_P
- C302 pad 1: /FPGA-01/1V0 -> /POWER/VSEN_P
- C303 pad 1: /FPGA-01/1V0 -> /POWER/VSEN_P
- C304 pad 1: /FPGA-01/1V0 -> /POWER/VSEN_P
- C38 pad 1: /POWER/VSEN_P -> /POWER/1V0_PRESH
- C42 pad 1: /POWER/VSEN_P -> /POWER/1V0_PRESH
- C46 pad 1: /POWER/VSEN_P -> /POWER/1V0_PRESH
- C49 pad 1: /POWER/VSEN_P -> /POWER/1V0_PRESH
- C52 pad 1: /POWER/VSEN_P -> /POWER/1V0_PRESH
- C55 pad 2: /POWER/VSEN_P -> /POWER/1V0_PRESH
- L3 pad 2: /POWER/VSEN_P -> /POWER/1V0_PRESH
- R165 pad 1: /FPGA-01/1V0 -> /POWER/VSEN_P
- R165 pad 2: /POWER/VSEN_P -> /POWER/1V0_PRESH
- U10 pad F10: /FPGA-01/1V0 -> /POWER/VSEN_P
- U10 pad F8: /FPGA-01/1V0 -> /POWER/VSEN_P
- U10 pad G11: /FPGA-01/1V0 -> /POWER/VSEN_P
- U10 pad G7: /FPGA-01/1V0 -> /POWER/VSEN_P
- U10 pad G9: /FPGA-01/1V0 -> /POWER/VSEN_P
- U10 pad H8: /FPGA-01/1V0 -> /POWER/VSEN_P
- U10 pad J11: /FPGA-01/1V0 -> /POWER/VSEN_P
- U10 pad J7: /FPGA-01/1V0 -> /POWER/VSEN_P
- U10 pad K8: /FPGA-01/1V0 -> /POWER/VSEN_P
- U10 pad L11: /FPGA-01/1V0 -> /POWER/VSEN_P
- U10 pad L7: /FPGA-01/1V0 -> /POWER/VSEN_P
- U10 pad M10: /FPGA-01/1V0 -> /POWER/VSEN_P
- U10 pad M8: /FPGA-01/1V0 -> /POWER/VSEN_P
- U10 pad N11: /FPGA-01/1V0 -> /POWER/VSEN_P
- U10 pad N7: /FPGA-01/1V0 -> /POWER/VSEN_P
- U10 pad N9: /FPGA-01/1V0 -> /POWER/VSEN_P
- U11 pad F10: /FPGA-01/1V0 -> /POWER/VSEN_P
- U11 pad F8: /FPGA-01/1V0 -> /POWER/VSEN_P
- U11 pad G11: /FPGA-01/1V0 -> /POWER/VSEN_P
- U11 pad G7: /FPGA-01/1V0 -> /POWER/VSEN_P
- U11 pad G9: /FPGA-01/1V0 -> /POWER/VSEN_P
- U11 pad H8: /FPGA-01/1V0 -> /POWER/VSEN_P
- U11 pad J11: /FPGA-01/1V0 -> /POWER/VSEN_P
- U11 pad J7: /FPGA-01/1V0 -> /POWER/VSEN_P
- U11 pad K8: /FPGA-01/1V0 -> /POWER/VSEN_P
- U11 pad L11: /FPGA-01/1V0 -> /POWER/VSEN_P
- U11 pad L7: /FPGA-01/1V0 -> /POWER/VSEN_P
- U11 pad M10: /FPGA-01/1V0 -> /POWER/VSEN_P
- U11 pad M8: /FPGA-01/1V0 -> /POWER/VSEN_P
- U11 pad N11: /FPGA-01/1V0 -> /POWER/VSEN_P
- U11 pad N7: /FPGA-01/1V0 -> /POWER/VSEN_P
- U11 pad N9: /FPGA-01/1V0 -> /POWER/VSEN_P
Routing:
- net /FPGA-01/1V0: track 101.2 -> 0.00 mm, vias 72 -> 0
- net /POWER/VSEN_P: track 45.4 -> 139.4 mm, vias 2 -> 74
- net GND: track 530.9 -> 503.5 mm, vias 808 -> 834
- net /PCIE/12V: track 319.8 -> 315.5 mm, vias 27 -> 25
- net /POWER/PGOOD_3V3: track 75.1 -> 78.6 mm
- net /FPGA-01/FPGA1_MISO: track 22.1 -> 20.6 mm
- net Net-(D25-A): track 3.86 -> 2.42 mm
- net /Audio_IN-OUT/3V3: track 341.5 -> 342.3 mm, vias 222 -> 223
- net Net-(U10A-IO_L2P_T0_AD8P_15): track 12.3 -> 11.6 mm
- net Net-(U3B-PVIN): track 6.00 -> 5.72 mm, vias 26 -> 22
- added copper zone on F.Cu, net /POWER/1V0_PRESH
- added copper zone on B.Cu, net /POWER/VSEN_P
- added copper zone on In1.Cu, net /POWER/VSEN_P
- added copper zone on In5.Cu, net /POWER/VSEN_P
- added copper zone on In6.Cu, net /POWER/VSEN_P
- added copper zone on In1.Cu, net GND
- removed copper zone on B.Cu, net /FPGA-01/1V0
- removed copper zone on F.Cu, net /FPGA-01/1V0
- removed copper zone on In1.Cu, net /FPGA-01/1V0
Other:
- board text added: "ECU Debug"
- board text added: "ECU JTAG"
- board text removed: "0"
- board text removed: "0 mm"
- board text removed: "0.01 mm"
- board text removed: "0.0152 mm"
- board text removed: "0.02"
- board text removed: "0.035 mm"
- board text removed: "0.1000 mm / 0.1270 mm"
- board text removed: "0.1164 mm"
- board text removed: "0.1500 mm"
- board text removed: "0.152 mm"
- board text removed: "0.3 mm"
- board text removed: "1"
- board text removed: "1.6180 mm"
- board text removed: "167.2300 mm x 95.4213 mm"
- board text removed: "3.3"
- board text removed: "4.5"
- board text removed: "8"
- board text removed: "B.Cu"
- board text removed: "B.Mask"
- board text removed: "B.Paste"
- board text removed: "B.Silkscreen"
- board text removed: "BOARD CHARACTERISTICS"
- board text removed: "Board Thickness:"
- board text removed: "Board overall dimensions:"
- board text removed: "Bottom Silk Screen"
- board text removed: "Bottom Solder Mask"
- board text removed: "Bottom Solder Paste"
- board text removed: "Castellated pads:"
- board text removed: "Color"
- board text removed: "Copper Finish:"
- board text removed: "Copper Layer Count:"
- board text removed: "Dielectric"
- board text removed: "Edge card connectors:"
- board text removed: "Epsilon R"
- board text removed: "F.Cu"
- board text removed: "F.Mask"
- board text removed: "F.Paste"
- board text removed: "F.Silkscreen"
- board text removed: "FR4"
- board text removed: "Impedance Control:"
- board text removed: "In1.Cu"
- board text removed: "In2.Cu"
- board text removed: "In3.Cu"
- board text removed: "In4.Cu"
- board text removed: "In5.Cu"
- board text removed: "In6.Cu"
- board text removed: "Layer Name"
- board text removed: "Loss Tangent"
- board text removed: "Material"
- board text removed: "Min hole diameter:"
- board text removed: "Min track/spacing:"
- board text removed: "No"
- board text removed: "None"
- board text removed: "Not specified"
- board text removed: "Plated Board Edge:"
- board text removed: "Thickness (mm)"
- board text removed: "Top Silk Screen"
- board text removed: "Top Solder Mask"
- board text removed: "Top Solder Paste"
- board text removed: "Type"
- board text removed: "Yes"
- board text removed: "copper"
- board text removed: "core"
- board text removed: "prepreg"
- board text removed: "uC Debug"
- board text removed: "uC JTAG"
