File: RASBB/Hardware/Rev.C/Design/Audio_IN-OUT.kicad_sch (KiCad schematic)
At the start: 20 parts, among them J12 AudioJack4, U8 LM386, U9 LM321

Commit message: RevC_06
Parts:
- C165: Mfr. Part #  UUD1A221MCL1GS -> (none)
- J12: value AudioJack4 -> AUDIO
- R123: LCSC Part # C227390 -> C163933; Mfr. Part #  WR06X5102FTL -> (none)
- U8: Mfr. Part #  LM386D -> (none)
Connections:
- net +3V3 renamed 3V3
- net +5V renamed 5V0
