File: RASBB/Hardware/Rev.C/Design/Config-SPI FLASH.kicad_sch (KiCad schematic)
At the start: 14 parts, among them IC5 S25FL128LAGMFI010, IC6 TS3A5018DBQR, IC7 S25FL128LAGMFI010, IC8 TS3A5018DBQR

Commit message: RevC_06
Parts:
- R196, R197, R198, R199, R53, R55: LCSC Part # C105871 -> C163826; Mfr. Part # RC0402FR-074K7L -> WR04X4701FTL
Connections:
- net +3V3 renamed 3V3
- net CS_Flash_FPGA2 renamed CS_FLASH_FPGA2
- net CS_Flash_uC renamed CS_FLASH_uC
- net SCK_Flash_FPGA2 renamed SCK_FLASH_FPGA2
- net SCK_Flash_uC renamed SCK_FLASH_uC
- net SI_Flash_FPGA2 renamed SI_FLASH_FPGA2
- net SI_Flash_uC renamed SI_FLASH_uC
- net SO_Flash_FPGA2 renamed SO_FLASH_FPGA2
- net SO_Flash_uC renamed SO_FLASH_uC
