File: RASBB/Hardware/Rev.C/Design/Ethernet_FPGA.kicad_sch (KiCad schematic)
At the start: 53 parts, among them J2 HR911196AE, U12 RTL8211E-VB-CG, X1 OT2EL4C4JI-111OLP-50M

Commit message: RevC_06
Parts:
- C62: Mfr. Part #  GRM21BR61A476ME15L -> (none)
- C73: Mfr. Part #   FV55X104K202EGG -> (none)
- C74: value tbd -> 1nF
- D4, D5: Mfr. Part #   DF1501S-T -> (none)
- J2: value HR911196AE -> ETH_1G; LCSC Part #   C5149194 -> (none); Mfr. Part #   HR911196AE -> (none)
- L7: LCSC Part #   C486337 -> (none); Mfr. Part # microgate MGFL3216F2R2MT-LF -> MGFL3216F2R2MT-LF; Mfr. Part #   MGFL3216F2R2MT-LF -> (none)
- L8: LCSC Part #   C88999 -> (none); Mfr. Part #   BLM41PG102SN1L -> (none)
- R107, R57, R58, R59, R60, R61, R62, R74, R76: value 4.7K -> 4K7; Mfr. Part #  WR04X4701FTL -> (none)
- R203: LCSC Part # C114768 -> C145071; Mfr. Part #  RC0402FR-072K49L -> (none)
- R210, R82: LCSC Part #   C880838 -> (none); Mfr. Part #   SR04X271JTL -> (none)
- R78, R79, R80, R81: LCSC Part #   C2074227 -> (none); Mfr. Part #   ESR03EZPF75R0 -> (none)
- TP4: now fitted
- U12: Mfr. Part #  RTL8211E-VB-CG -> (none)
Connections:
- net +3V3 renamed 3V3
Other:
- moved on the sheet: C352, C357, C358, C359, C360, C361, C362, C363, C364, C62, C63, C64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
