File: RASBB/Hardware/Rev.C/Design/Ethernet_uC.kicad_sch (KiCad schematic)
At the start: 61 parts, among them IC14 LAN8742AI-CZ-TR, IC15 DS90LV028AQDQFRQ1, J14 636101112001, J19 HC-WK88-H16-DB, T1 15FB-30NL, Y3 25MHz

Commit message: RevC_06
Parts:
- C170: Mfr. Part #  GRM21BR61A476ME15L -> (none)
- C181: LCSC Part #   C303946 -> (none); Mfr. Part #   1206B102K202CT -> (none)
- C183, C322: value tbd -> 1nF
- D10: LCSC Part #   C445539 -> (none)
- D26: Mfr. Part #   DF1501S-T -> (none)
- IC14: LCSC Part #   C621425 -> (none); Mfr. Part #   LAN8742AI-CZ-TR -> (none)
- IC15: Manufacturer_Part_Number DS90LV028AQDQFRQ1 -> (none)
- J14: value 636101112001 -> SYNC_40MHZ; Part Number 636101112001 -> (none)
- J19: value HC-WK88-H16-DB -> ETH_100M_POE; MF Hong Cheng -> (none)
- L11: LCSC Part #   C88999 -> (none); Mfr. Part #   BLM41PG102SN1L -> (none)
- R134: LCSC Part #   C168199 -> (none); Mfr. Part #   WR04X1212FTL -> (none)
- R143: Mfr. Part #   RCS06030000Z0EC -> (none)
- R144, R145: LCSC Part #   C2074227 -> (none); Mfr. Part #   ESR03EZPF75R0 -> (none)
- R186, R83: LCSC Part #   C880838 -> (none); Mfr. Part #   SR04X271JTL -> (none)
Connections:
- net +3V3 renamed 3V3

Commit message: REV.C production data
Parts:
- removed C183: 1nF, Capacitor_SMD:C_1206_3216Metric, symbol Device:C_Small
Changed lines of the file:
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@@
 	(title_block
 		(title "RASBB")
-		(date "2026-09-27")
-		(rev "C.6")
+		(date "2026-09-29")
+		(rev "C")
 		(company "Mina Daneshpajouh")
 	)
@@
 					(unit 1)
 				)
-			)
-		)
-	)
-	(symbol
-		(lib_id "Device:C_Small")
-		(at 335.28 139.7 0)
-		(unit 1)
-		(body_style 1)
-		(exclude_from_sim no)
-		(in_bom yes)
-		(on_board yes)
-		(in_pos_files yes)
-		(dnp yes)
-		(property "Reference" "C183"
-			(at 336.55 138.43 0)
-			(show_name no)
-			(do_not_autoplace no)
-			(effects
-				(font
-					(size 1.27 1.27)
-				)
-				(justify left)
-			)
-		)
-		(property "Value" "1nF"
-			(at 336.55 140.97 0)
-			(show_name no)
-			(do_not_autoplace no)
-			(effects
-				(font
-					(size 1.27 1.27)
-				)
-				(justify left)
-			)
-		)
-		(property "Footprint" "Capacitor_SMD:C_1206_3216Metric"
-			(at 335.28 139.7 0)
-			(hide yes)
-			(show_name no)
-			(do_not_autoplace no)
-			(effects
-				(font
-					(size 1.27 1.27)
-				)
-			)
-		)
-		(property "Datasheet" ""
-			(at 335.28 139.7 0)
-			(hide yes)
-			(show_name no)
-			(do_not_autoplace no)
-			(effects
-				(font
-					(size 1.27 1.27)
-				)
-			)
-		)
-		(property "Description" "CAP, CER, 1nF, 2kV, 10%, X7R, 1210"
-			(at 335.28 139.7 0)
-			(hide yes)
-			(show_name no)
-			(do_not_autoplace no)
-			(effects
-				(font
-					(size 1.27 1.27)
-				)
-			)
-		)
-		(pin "1"
-		)
-		(pin "2"
-		)
-		(instances
-			(project "RASBB"
-				(path "/f6a5c334-5ee5-4dc9-84f1-7866383a3347/1cb570e6-5b4c-4568-b1cb-9ef0ed6103b4"
-					(reference "C183")
-					(unit 1)
-				)
