File: RASBB/Hardware/Rev.C/Design/FPGA01.kicad_sch (KiCad schematic)
At the start: 0 parts

Commit message: RevC_06
Other:
- sheet BANK35 ports: added 1V8; removed none
- sheet FPGA_POWER ports: added 1V0; removed none
