File: RASBB/Hardware/Rev.C/Design/FPGA1_BANK14-15.kicad_sch (KiCad schematic)
At the start: 27 parts, among them U10 XC7A100T-CSG324

Commit message: RevC_06
Parts:
- C188: Mfr. Part #  GRM21BR61A476ME15L -> (none)
- C233, C234, C235, C236, C239, C241, C242, C243, C244, C245, C251, C252, C253, C254, C255, C257: Mfr. Part # GRT155R71A474KE01D -> GRM155R71C474KE01D
- C246, C247, C249, C250: LCSC Part #  C77004 -> (none)
- C248: Mfr. Part #  GRM31CR61A107MEA8L -> (none)
- D24: LCSC Part #   C5355434 -> (none); Mfr. Part #   A-SP192GS1D-C01-4T -> (none)
- D25: LCSC Part #   C19171301 -> (none); Mfr. Part #   A-SP192DGHC-C01-4T -> (none)
- U10: Mfr. Part #  XC7A100T-2CSG324I -> (none)
Other:
- moved on the sheet: C188, C233, C234, C235, C236, C239, C241, C242, C243, C244, C245, C246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
