File: RASBB/Hardware/Rev.C/Design/FPGA1_BANK16-34.kicad_sch (KiCad schematic)
At the start: 11 parts, among them U10 XC7A100T-CSG324

Commit message: RevC_06
Parts:
- C223, C227, C228: LCSC Part #  C77004 -> (none)
- C224, C229, C230, C231, C232, C75: Mfr. Part # GRT155R71A474KE01D -> GRM155R71C474KE01D
- C226: Mfr. Part #  GRM31CR61A107MEA8L -> (none)
- U10: Mfr. Part #  XC7A100T-2CSG324I -> (none)
Other:
- moved on the sheet: C223, C224
