File: RASBB/Hardware/Rev.C/Design/FPGA1_BANK35.kicad_sch (KiCad schematic)
At the start: 17 parts, among them J16 Conn_01x02_Pin, U10 XC7A100T-CSG324, X3 OT2EL4C4JI-111OLP-50M

Commit message: RevC_06
Parts:
- C182, C225, C261, C262, C263, C264, C265: Mfr. Part # GRT155R71A474KE01D -> GRM155R71C474KE01D
- C192: Mfr. Part #  GRM21BR61A476ME15L -> (none)
- C266, C267: LCSC Part #  C77004 -> (none)
- J16: value Conn_01x02_Pin -> FPGA1_CLK_OUT
- U10: Mfr. Part #  XC7A100T-2CSG324I -> (none)
Connections:
- net +1V8 renamed 1V8
