File: RASBB/Hardware/Rev.C/Design/FPGA1_DDR3.kicad_sch (KiCad schematic)
At the start: 32 parts, among them IC9 MT41K128M16JT-107:K

Commit message: RevC_06
Parts:
- C89, C92: Mfr. Part # GRT155R71A474KE01D -> GRM155R71C474KE01D
- R85, R86: LCSC Part # C105871 -> C163826; Mfr. Part # RC0402FR-074K7L -> WR04X4701FTL
