File: RASBB/Hardware/Rev.C/Design/FPGA1_PWR.kicad_sch (KiCad schematic)
At the start: 30 parts, among them U10 XC7A100T-CSG324

Commit message: RevC_06
Parts:
- C184: Mfr. Part #  GRM21BR61A476ME15L -> (none)
- C185, C189, C190, C191, C193, C194, C196, C197, C200, C201, C203, C205, C207, C209: Mfr. Part # GRT155R71A474KE01D -> GRM155R71C474KE01D
- C198, C218, C219, C220: Mfr. Part #  GRM31CR61A107MEA8L -> (none)
- C206, C208, C210, C211, C212, C213, C214, C215, C216, C217: LCSC Part #  C77004 -> (none)
- U10: Mfr. Part #  XC7A100T-2CSG324I -> (none)
Connections:
- net VCCBRAM: no longer C190.1, C194.1, C198.1
- net +1V0 renamed 1V0
- net 1V0: now also C190.1, C194.1, C198.1
