File: RASBB/Hardware/Rev.C/Design/FPGA2_BANK14-15.kicad_sch (KiCad schematic)
At the start: 20 parts, among them U11 XC7A100T-CSG324

Commit message: RevC_06
Parts:
- C195, C332: Mfr. Part #  GRM31CR61A107MEA8L -> (none)
- C326, C327, C328, C329, C335, C336, C337, C338: Mfr. Part # GRT155R71A474KE01D -> GRM155R71C474KE01D
- C330, C331, C333, C334: LCSC Part #  C77004 -> (none)
- D22: LCSC Part #   C19171301 -> (none); Mfr. Part #   A-SP192DGHC-C01-4T -> (none)
- D23: LCSC Part #   C5355434 -> (none); Mfr. Part #   A-SP192GS1D-C01-4T -> (none)
- U11: Mfr. Part #  XC7A100T-2CSG324I -> (none)
