File: RASBB/Hardware/Rev.C/Design/FPGA2_BANK16-34.kicad_sch (KiCad schematic)
At the start: 11 parts, among them U11 XC7A100T-CSG324

Commit message: RevC_06
Parts:
- C307, C311, C312: LCSC Part #  C77004 -> (none)
- C308, C313, C314, C315, C316: Mfr. Part # GRT155R71A474KE01D -> GRM155R71C474KE01D
- C310: Mfr. Part #  GRM31CR61A107MEA8L -> (none)
- U11: Mfr. Part #  XC7A100T-2CSG324I -> (none)
Changed lines of the file:
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@@
 	(title_block
 		(title "RASBB")
-		(date "2026-09-20")
-		(rev "C")
+		(date "2026-09-27")
+		(rev "C.6")
 		(company "Mina Daneshpajouh")
 	)
@@
 			(width 0)
 			(type default)
+			(color 150 0 200 1)
 		)
 	)
@@
 			(width 0)
 			(type default)
+			(color 0 0 0 1)
 		)
 	)
@@
 			(width 0)
 			(type default)
+			(color 150 0 200 1)
 		)
 	)
@@
 			(width 0)
 			(type default)
+			(color 150 0 200 1)
 		)
 	)
@@
 			(width 0)
 			(type default)
+			(color 150 0 200 1)
 		)
 	)
@@
 			(width 0)
 			(type default)
+			(color 0 0 0 1)
 		)
 	)
@@
 			(width 0)
 			(type default)
+			(color 0 0 0 1)
 		)
 	)
@@
 			(width 0)
 			(type default)
+			(color 0 0 0 1)
 		)
 	)
@@
 			(width 0)
 			(type default)
+			(color 150 0 200 1)
 		)
 	)
@@
 			(width 0)
 			(type default)
+			(color 150 0 200 1)
 		)
 	)
@@
 			(width 0)
 			(type default)
+			(color 150 0 200 1)
 		)
 	)
@@
 			(width 0)
 			(type default)
+			(color 150 0 200 1)
 		)
 	)
@@
 			(width 0)
 			(type default)
+			(color 150 0 200 1)
 		)
 	)
@@
 			(width 0)
 			(type default)
+			(color 150 0 200 1)
 		)
 	)
@@
 			(width 0)
 			(type default)
+			(color 150 0 200 1)
 		)
 	)
@@
 			(width 0)
 			(type default)
+			(color 150 0 200 1)
 		)
 	)
@@
 			(width 0)
 			(type default)
+			(color 0 0 0 1)
 		)
 	)
@@
 			(width 0)
 			(type default)
+			(color 150 0 200 1)
 		)
 	)
@@
 			(width 0)
 			(type default)
+			(color 150 0 200 1)
 		)
 	)
@@
 			(width 0)
 			(type default)
+			(color 150 0 200 1)
 		)
 	)
@@
 			(width 0)
 			(type default)
+			(color 150 0 200 1)
 		)
 	)
@@
 			(width 0)
 			(type default)
+			(color 150 0 200 1)
 		)
 	)
@@
 			(width 0)
 			(type default)
+			(color 150 0 200 1)
 		)
 	)
@@
 			(width 0)
 			(type default)
+			(color 150 0 200 1)
 		)
 	)
@@
 			(width 0)
 			(type default)
+			(color 150 0 200 1)
 		)
 	)
@@
 			(width 0)
 			(type default)
+			(color 150 0 200 1)
 		)
 	)
@@
 			(width 0)
 			(type default)
+			(color 150 0 200 1)
 		)
 	)
@@
 			)
 		)
-		(property "LCSC Part # " "C77004"
-			(at 74.93 62.23 0)
-			(hide yes)
-			(show_name no)
-			(do_not_autoplace no)
-			(effects
-				(font
-					(size 1.27 1.27)
-				)
-			)
-		)
 		(property "LCSC Part #" "C77004"
 			(at 74.93 62.23 0)
@@
 			)
 		)
-		(property "Mfr. Part #" "GRT155R71A474KE01D "
+		(property "Mfr. Part #" "GRM155R71C474KE01D"
 			(at 270.51 62.23 0)
 			(hide yes)
@@
 			)
 		)
-		(property "Mfr. Part # " "GRM31CR61A107MEA8L"
-			(at 231.14 62.23 0)
-			(hide yes)
-			(show_name no)
-			(do_not_autoplace no)
-			(effects
-				(font
-					(size 1.27 1.27)
-				)
-			)
-		)
 		(property "LCSC Part #" "C883598"
 			(at 231.14 62.23 0)
@@
 			)
 		)
-		(property "Mfr. Part #" "GRT155R71A474KE01D "
+		(property "Mfr. Part #" "GRM155R71C474KE01D"
 			(at 83.82 62.23 0)
 			(hide yes)
@@
 			)
 		)
-		(property "Mfr. Part #" "GRT155R71A474KE01D "
+		(property "Mfr. Part #" "GRM155R71C474KE01D"
 			(at 279.4 62.23 0)
 			(hide yes)
@@
 			)
 		)
-		(property "LCSC Part # " "C77004"
-			(at 241.3 62.23 0)
-			(hide yes)
-			(show_name no)
-			(do_not_autoplace no)
-			(effects
-				(font
-					(size 1.27 1.27)
-				)
-			)
-		)
 		(property "LCSC Part #" "C77004"
 			(at 241.3 62.23 0)
@@
 			)
 		)
-		(property "LCSC Part # " "C77004"
-			(at 251.46 62.23 0)
-			(hide yes)
-			(show_name no)
-			(do_not_autoplace no)
-			(effects
-				(font
-					(size 1.27 1.27)
-				)
-			)
-		)
 		(property "LCSC Part #" "C77004"
 			(at 251.46 62.23 0)
@@
 			)
 		)
-		(property "Mfr. Part # " "XC7A100T-2CSG324I "
-			(at 179.07 132.08 0)
-			(hide yes)
-			(show_name no)
-			(do_not_autoplace no)
-			(effects
-				(font
-					(size 1.27 1.27)
-				)
-			)
-		)
 		(property "LCSC Part #" "C1521791"
 			(at 179.07 132.08 0)
@@
 			)
 		)
-		(property "Mfr. Part #" "GRT155R71A474KE01D "
+		(property "Mfr. Part #" "GRM155R71C474KE01D"
 			(at 260.35 62.23 0)
 			(hide yes)
@@
 			)
 		)
-		(property "Mfr. Part #" "GRT155R71A474KE01D "
+		(property "Mfr. Part #" "GRM155R71C474KE01D"
 			(at 287.02 62.23 0)
 			(hide yes)
