File: RASBB/Hardware/Rev.C/Design/FPGA2_BANK35.kicad_sch (KiCad schematic)
At the start: 14 parts, among them J18 Conn_01x02_Pin, U11 XC7A100T-CSG324, X4 OT2EL4C4JI-111OLP-50M

Commit message: RevC_06
Parts:
- C199: Mfr. Part #  GRM31CR61A107MEA8L -> (none)
- C346, C347, C348, C349: Mfr. Part # GRT155R71A474KE01D -> GRM155R71C474KE01D
- C351: LCSC Part #  C77004 -> (none)
- J18: value Conn_01x02_Pin -> FPGA2_CLK_OUT
- U11: Mfr. Part #  XC7A100T-2CSG324I -> (none)
Connections:
- net +3V3 renamed 3V3
Changed lines of the file:
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@@
 	(title_block
 		(title "RASBB")
-		(date "2026-09-20")
-		(rev "C")
+		(date "2026-09-27")
+		(rev "C.6")
 		(company "Mina Daneshpajouh")
 	)
@@
 			(width 0)
 			(type default)
+			(color 220 0 0 1)
 		)
 	)
@@
 			(width 0)
 			(type default)
+			(color 220 0 0 1)
 		)
 	)
@@
 			(width 0)
 			(type default)
+			(color 220 0 0 1)
 		)
 	)
@@
 			(width 0)
 			(type default)
+			(color 220 0 0 1)
 		)
 	)
@@
 			(width 0)
 			(type default)
+			(color 220 0 0 1)
 		)
 	)
@@
 			(width 0)
 			(type default)
+			(color 220 0 0 1)
 		)
 	)
@@
 			(width 0)
 			(type default)
+			(color 220 0 0 1)
 		)
 	)
@@
 			(width 0)
 			(type default)
+			(color 220 0 0 1)
 		)
 	)
@@
 			(width 0)
 			(type default)
+			(color 220 0 0 1)
 		)
 	)
@@
 			(width 0)
 			(type default)
+			(color 220 0 0 1)
 		)
 	)
@@
 			(width 0)
 			(type default)
+			(color 220 0 0 1)
 		)
 	)
@@
 			(width 0)
 			(type default)
+			(color 220 0 0 1)
 		)
 	)
@@
 			(width 0)
 			(type default)
+			(color 220 0 0 1)
 		)
 	)
@@
 			(width 0)
 			(type default)
+			(color 220 0 0 1)
 		)
 	)
@@
 			(width 0)
 			(type default)
+			(color 220 0 0 1)
 		)
 	)
@@
 			(width 0)
 			(type default)
+			(color 220 0 0 1)
 		)
 	)
@@
 			(width 0)
 			(type default)
+			(color 220 0 0 1)
 		)
 	)
@@
 			(width 0)
 			(type default)
+			(color 220 0 0 1)
 		)
 	)
@@
 			(width 0)
 			(type default)
+			(color 220 0 0 1)
 		)
 	)
@@
 			(width 0)
 			(type default)
+			(color 220 0 0 1)
 		)
 	)
@@
 			(width 0)
 			(type default)
+			(color 220 0 0 1)
 		)
 	)
@@
 		)
 	)
+	(hierarchical_label "3V3"
+		(shape input)
+		(at 87.63 125.73 90)
+		(effects
+			(font
+				(size 1.27 1.27)
+			)
+			(justify left)
+		)
+	)
 	(hierarchical_label "F2_B35_A1"
 		(shape output)
@@
 			)
 		)
-		(property "Mfr. Part #" "GRT155R71A474KE01D "
+		(property "Mfr. Part #" "GRM155R71C474KE01D"
 			(at 118.11 64.77 0)
 			(hide yes)
@@
 			)
 		)
-		(property "Mfr. Part #" "GRT155R71A474KE01D "
+		(property "Mfr. Part #" "GRM155R71C474KE01D"
 			(at 125.73 64.77 0)
 			(hide yes)
@@
 			)
 		)
-		(property "LCSC Part # " "C77004"
-			(at 163.83 64.77 0)
-			(hide yes)
-			(show_name no)
-			(do_not_autoplace no)
-			(effects
-				(font
-					(size 1.27 1.27)
-				)
-			)
-		)
 		(property "LCSC Part #" "C77004"
 			(at 163.83 64.77 0)
@@
 			)
 		)
-		(property "Mfr. Part #" "GRT155R71A474KE01D "
+		(property "Mfr. Part #" "GRM155R71C474KE01D"
 			(at 143.51 64.77 0)
 			(hide yes)
@@
 			)
 		)
-		(property "Mfr. Part # " "GRM31CR61A107MEA8L"
-			(at 104.14 64.77 0)
-			(hide yes)
-			(show_name no)
-			(do_not_autoplace no)
-			(effects
-				(font
-					(size 1.27 1.27)
-				)
-			)
-		)
 		(property "LCSC Part #" "C883598"
 			(at 104.14 64.77 0)
@@
 			)
 		)
-		(property "Description" "Resistor, small symbol"
+		(property "Description" "62.5mW Thick Film Resistors 50V ±100ppm/℃ ±1% 49.9Ω 0402 Chip Resistor - Surface Mount ROHS"
 			(at 87.63 130.81 0)
 			(hide yes)
@@
 	)
 	(symbol
-		(lib_id "power:+3.3V")
-		(at 87.63 125.73 0)
-		(unit 1)
-		(body_style 1)
-		(exclude_from_sim no)
-		(in_bom yes)
-		(on_board yes)
-		(in_pos_files yes)
-		(dnp no)
-		(property "Reference" "#PWR0236"
-			(at 87.63 129.54 0)
-			(hide yes)
-			(show_name no)
-			(do_not_autoplace no)
-			(effects
-				(font
-					(size 1.27 1.27)
-				)
-			)
-		)
-		(property "Value" "+3V3"
-			(at 80.772 124.968 0)
-			(show_name no)
-			(do_not_autoplace no)
-			(effects
-				(font
-					(size 1.27 1.27)
-				)
-				(justify left)
-			)
-		)
-		(property "Footprint" ""
-			(at 87.63 125.73 0)
-			(hide yes)
-			(show_name no)
-			(do_not_autoplace no)
-			(effects
-				(font
-					(size 1.27 1.27)
-				)
-			)
-		)
-		(property "Datasheet" ""
-			(at 87.63 125.73 0)
-			(hide yes)
-			(show_name no)
-			(do_not_autoplace no)
-			(effects
-				(font
-					(size 1.27 1.27)
-				)
-			)
-		)
-		(property "Description" "Power symbol creates a global label with name \"+3.3V\""
-			(at 87.63 125.73 0)
-			(hide yes)
-			(show_name no)
-			(do_not_autoplace no)
-			(effects
-				(font
-					(size 1.27 1.27)
-				)
-			)
-		)
-		(pin "1"
-		)
-		(instances
-			(project "RASBB"
-				(path "/f6a5c334-5ee5-4dc9-84f1-7866383a3347/1039afa1-78bb-4140-9ce0-f929b7009905/07a5a2f3-3ce6-4945-b18c-18d4cab18b87"
-					(reference "#PWR0236")
-					(unit 1)
-				)
-			)
-		)
-	)
-	(symbol
 		(lib_id "Device:R_Small")
 		(at 123.19 142.24 90)
@@
 			)
 		)
-		(property "Description" "Resistor, small symbol"
+		(property "Description" "62.5mW Thick Film Resistors 50V ±100ppm/℃ ±1% 49.9Ω 0402 Chip Resistor - Surface Mount ROHS"
 			(at 123.19 142.24 0)
 			(hide yes)
@@
 			)
 		)
-		(property "Value" "Conn_01x02_Pin"
+		(property "Value" "FPGA2_CLK_OUT"
 			(at 107.315 149.86 0)
 			(show_name no)
@@
 			)
 		)
-		(property "Mfr. Part #" "GRT155R71A474KE01D "
+		(property "Mfr. Part #" "GRM155R71C474KE01D"
 			(at 134.62 64.77 0)
 			(hide yes)
@@
 			)
 		)
-		(property "Description" "Resistor, small symbol"
+		(property "Description" "62.5mW Thick Film Resistors 50V ±100ppm/℃ ±1% 49.9Ω 0402 Chip Resistor - Surface Mount ROHS"
 			(at 96.52 139.7 0)
 			(hide yes)
@@
 			)
 		)
-		(property "Mfr. Part # " "XC7A100T-2CSG324I "
-			(at 214.63 134.62 0)
-			(hide yes)
-			(show_name no)
-			(do_not_autoplace no)
-			(effects
-				(font
-					(size 1.27 1.27)
-				)
-			)
-		)
 		(property "LCSC Part #" "C1521791"
 			(at 214.63 134.62 0)
@@
 				)
 			)
+		)
+	)
+	(symbol
+		(lib_id "power:PWR_FLAG")
+		(at 58.42 124.46 0)
+		(unit 1)
+		(body_style 1)
+		(exclude_from_sim no)
+		(in_bom yes)
+		(on_board yes)
+		(in_pos_files yes)
+		(dnp no)
+		(fields_autoplaced yes)
+		(property "Reference" "#FLG017"
+			(at 58.42 122.555 0)
+			(hide yes)
+			(show_name no)
+			(do_not_autoplace no)
+			(effects
+				(font
+					(size 1.27 1.27)
+				)
+			)
+		)
+		(property "Value" "PWR_FLAG"
+			(at 58.42 119.38 0)
+			(hide yes)
+			(show_name no)
+			(do_not_autoplace no)
+			(effects
+				(font
+					(size 1.27 1.27)
+				)
+			)
+		)
+		(property "Footprint" ""
+			(at 58.42 124.46 0)
+			(hide yes)
+			(show_name no)
+			(do_not_autoplace no)
+			(effects
+				(font
+					(size 1.27 1.27)
+				)
+			)
+		)
+		(property "Datasheet" ""
+			(at 58.42 124.46 0)
+			(hide yes)
+			(show_name no)
+			(do_not_autoplace no)
+			(effects
+				(font
+					(size 1.27 1.27)
+				)
+			)
+		)
+		(property "Description" "Special symbol for telling ERC where power comes from"
+			(at 58.42 124.46 0)
+			(hide yes)
+			(show_name no)
+			(do_not_autoplace no)
+			(effects
+				(font
+					(size 1.27 1.27)
+				)
+			)
+		)
+		(pin "1"
+		)
+		(instances
+			(project "RASBB"
+				(path "/f6a5c334-5ee5-4dc9-84f1-7866383a3347/1039afa1-78bb-4140-9ce0-f929b7009905/07a5a2f3-3ce6-4945-b18c-18d4cab18b87"
+					(reference "#FLG017")
+					(unit 1)
+				)
+			)
