File: RASBB/Hardware/Rev.C/Design/FPGA2_PWR.kicad_sch (KiCad schematic)
At the start: 30 parts, among them U11 XC7A100T-CSG324

Commit message: RevC_06
Parts:
- C187: Mfr. Part #  GRM21BR61A476ME15L -> (none)
- C269, C273, C274, C275, C277, C278, C280, C281, C284, C285, C287, C289, C291, C293: Mfr. Part # GRT155R71A474KE01D -> GRM155R71C474KE01D
- C282, C302, C303, C304: Mfr. Part #  GRM31CR61A107MEA8L -> (none)
- C290, C292, C294, C295, C296, C297, C298, C299, C300, C301: LCSC Part #  C77004 -> (none)
- U11: Mfr. Part #  XC7A100T-2CSG324I -> (none)
Connections:
- net VCCBRAM: no longer C274.1, C278.1, C282.1
- net +1V0 renamed 1V0
- net 1V0: now also C274.1, C278.1, C282.1
