File: RASBB/Hardware/Rev.C/Design/HDMI.kicad_sch (KiCad schematic)
At the start: 21 parts, among them IC11 TPD12S016PWR, J3 HDMI-001A

Commit message: RevC_06
Parts:
- IC11: Mfr. Part #  TPD12S016PWR -> (none)
- J3: value HDMI-001A -> HDMI; Mfr. Part #  HDMI-001A -> (none)
- R212, R213, R214, R215, R216, R217, R218, R219: LCSC Part #   C880838 -> (none); Mfr. Part #   SR04X271JTL -> (none)
Connections:
- net +3V3 renamed 3V3
- net +5V renamed 5V0
Other:
- moved on the sheet: C122, C124
