File: RASBB/Hardware/Rev.C/Design/Interconnect.kicad_sch (KiCad schematic)
At the start: 13 parts, among them J5 FH12-50S-0.5SV

Commit message: RevC_06
Parts:
- J5: value FH12-50S-0.5SV -> ICON
- RN1, RN10, RN2, RN3, RN4, RN5, RN6, RN7, RN8, RN9: Manufacturer_Part_Number CAY10-330J4LF -> (none)
Connections:
- net +3V3 renamed 3V3
