File: RASBB/Hardware/Rev.C/Design/PCIE.kicad_sch (KiCad schematic)
At the start: 5 parts, among them J17 Conn_01x02_Pin, J4 X3157WS-98-9TV30

Commit message: RevC_06
Parts:
- removed R208, R209: 0, Resistor_SMD:R_1206_3216Metric, symbol Device:R
- added J6: Conn_01x03, Connector_PinHeader_2.54mm:PinHeader_1x03_P2.54mm_Vertical, symbol Connector_Generic:Conn_01x03
- J17: value Conn_01x02_Pin -> FE_3V3_MEAS
- J4: value X3157WS-98-9TV30 -> FRONTEND; Mfr. Part #  X3157WS-98-9TV30 -> (none)
- R185: Mfr. Part #   1206W4F0000T5E -> (none)
Connections:
- net at J4.A01, J4.A02, J4.A03: no longer J4.B01, J4.B02, J4.B03
- net +3V3 renamed 3V3
- new net: J4.B01, J4.B02, J4.B03, J6.2 (Pin_2)
- new net 12V: J6.3 (Pin_3)
- new net 5V0: J6.1 (Pin_1)
- no-connect marks 0 -> 2
