File: RASBB/Hardware/Rev.C/Design/POQWE.kicad_sch (KiCad schematic)
At the start: 112 parts, among them IC1 RT6365GSP, IC2 TPS56528DDAR, IC3 TPS563201DDCR, IC4 TPS56528DDAR, J1 PJ-002AH-SMT-TR, U1 SZMMSZ4702T1G, U2 SI2324DS-T1-GE3, U3 SIC453ED-T1-GE3, U4 JW5026

Commit message: RevC_06
Parts:
- added R220, R221, R222, R223: 0.005, Resistor_SMD:R_2512_6332Metric, symbol Device:R_Small
- C30, C32: Mfr. Part # GRT155R71A474KE01D -> GRM155R71C474KE01D
- C4: value 10uF -> 10uF, 100V; Mfr. Part #  C3216X6S2A106K160AC -> (none)
- C42, C46, C49, C52: Mfr. Part #  GRM21BR61A476ME15L -> (none)
- D1: Mfr. Part #  SDT5A60SA-13 -> (none)
- D2, D3: Mfr. Part #  VSSAF5L45HM3_A/H -> (none)
- D20, D21: LCSC Part #   C19171301 -> (none); Mfr. Part #   A-SP192DGHC-C01-4T -> (none)
- IC1: Mfr. Part #  RT6365GSP -> (none)
- J1: value PJ-002AH-SMT-TR -> DC_12V_IN
- L1: Mfr. Part #  0630CDMCDDS-100MC -> (none)
- L2: Mfr. Part #  SMDRS6028-150N -> (none)
- L3: Mfr. Part #  IHLP4040DZERR36M01 -> (none)
- L4, L5, L6: Mfr. Part #  IHLP2525EZER2R2M01 -> (none)
- R165: LCSC Part # C7419996 -> C7467241
- R25: Mfr. Part #  WR12X2492FTL -> (none)
- R26: Mfr. Part #  WR08X2493FTL -> (none)
- R27: LCSC Part # C227390 -> C163933; Mfr. Part #  WR06X5102FTL -> (none)
- R32, R44: LCSC Part # C384380 -> C4170964
- U1: Mfr. Part #  SZMMSZ4702T1G -> (none)
- U2: Mfr. Part #  SI2324DS-T1-GE3 -> (none)
- U4: Mfr. Part #  JW5026 -> (none)
- Z1: Mfr. Part #  MMSZ5255BT1G -> (none)
Connections:
- net 12V: now reaches F2.1, R211.2
- net 12V: now also R220.2, R221.2, R222.2, R223.2
- removed net +12V: C17.1, C18.1, C21.1, C22.1, C23.1, C24.1, C25.1, C26.1, C27.1, C28.1, C29.1, C31.1, C354.1, C355.1, C356.1, IC2.8 (VIN), IC3.3 (VIN), IC4.8 (VIN), R211.1, R36.2, R42.1, U3.1-3/34 (PVIN), U3.23 (VIN), U4.5 (VIN)
- net +1V0 renamed 1V0
- net +1V35 renamed 1V35
- net +1V8 renamed 1V8
- net +3V3 renamed 3V3
- net +5V renamed 5V0
- new net: C17.1, C18.1, C354.1, C355.1, C356.1, R211.1, R36.2, U3.1-3/34 (PVIN), U3.23 (VIN)
- new net: C29.1, R220.1, R42.1, U4.5 (VIN)
- new net: C21.1, C24.1, C27.1, IC2.8 (VIN), R222.1
- new net: C23.1, C26.1, C31.1, IC3.3 (VIN), R223.1
- new net: C22.1, C25.1, C28.1, IC4.8 (VIN), R221.1

Commit message: REV.C production data
Connections:
- net 1V0: now also U3.12 (VSEN+)
- net VSEN_P renamed 1V0_PRESH
- net 1V0_PRESH: no longer U3.12 (VSEN+)
Other:
- moved on the sheet: R165
Changed lines of the file:
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@@
 	(title_block
 		(title "RASBB")
-		(date "2026-09-27")
-		(rev "C.6")
+		(date "2026-09-29")
+		(rev "C")
 		(company "Mina Daneshpajouh")
 	)
@@
 	)
 	(junction
-		(at 755.65 208.28)
-		(diameter 0)
-		(color 0 0 0 0)
-	)
-	(junction
 		(at 505.46 256.54)
 		(diameter 0)
@@
 	)
 	(junction
+		(at 773.43 208.28)
+		(diameter 0)
+		(color 0 0 0 0)
+	)
+	(junction
 		(at 646.43 339.09)
 		(diameter 0)
@@
 	(wire
 		(pts
+			(xy 773.43 208.28) (xy 778.51 208.28)
+		)
+		(stroke
+			(width 0)
+			(type default)
+			(color 128 128 128 1)
+		)
+	)
+	(wire
+		(pts
 			(xy 746.76 302.26) (xy 746.76 314.96)
 		)
@@
 	(wire
 		(pts
-			(xy 755.65 208.28) (xy 765.81 208.28)
-		)
-		(stroke
-			(width 0)
-			(type default)
-		)
-	)
-	(wire
-		(pts
 			(xy 453.39 104.14) (xy 445.77 104.14)
 		)
@@
 	(wire
 		(pts
-			(xy 770.89 208.28) (xy 778.51 208.28)
+			(xy 760.73 208.28) (xy 773.43 208.28)
 		)
 		(stroke
@@
 	(wire
 		(pts
-			(xy 755.65 238.76) (xy 755.65 208.28)
-		)
-		(stroke
-			(width 0)
-			(type default)
-		)
-	)
-	(wire
-		(pts
 			(xy 688.34 107.95) (xy 693.42 107.95)
 		)
@@
 	(wire
 		(pts
-			(xy 740.41 208.28) (xy 755.65 208.28)
+			(xy 760.73 208.28) (xy 773.43 208.28)
 		)
 		(stroke
@@
 	(wire
 		(pts
+			(xy 740.41 208.28) (xy 755.65 208.28)
+		)
+		(stroke
+			(width 0)
+			(type default)
+		)
+	)
+	(wire
+		(pts
 			(xy 693.42 107.95) (xy 693.42 111.76)
 		)
@@
 	(wire
 		(pts
+			(xy 740.41 205.74) (xy 740.41 208.28)
+		)
+		(stroke
+			(width 0)
+			(type default)
+		)
+	)
+	(wire
+		(pts
 			(xy 297.18 259.08) (xy 251.46 259.08)
 		)
@@
 	(wire
 		(pts
-			(xy 681.99 238.76) (xy 755.65 238.76)
+			(xy 681.99 238.76) (xy 773.43 238.76)
 		)
 		(stroke
@@
 	(wire
 		(pts
+			(xy 773.43 238.76) (xy 773.43 208.28)
+		)
+		(stroke
+			(width 0)
+			(type default)
+		)
+	)
+	(wire
+		(pts
 			(xy 208.28 278.13) (xy 215.9 278.13)
 		)
@@
 		)
 	)
+	(label "1V0_PRESH"
+		(at 740.41 208.28 0)
+		(effects
+			(font
+				(size 1.27 1.27)
+			)
+			(justify left bottom)
+		)
+	)
 	(label "PGOOD_3V3"
 		(at 621.03 453.39 0)
@@
 	(symbol
 		(lib_id "power:PWR_FLAG")
-		(at 770.89 208.28 0)
+		(at 773.43 208.28 0)
 		(unit 1)
 		(body_style 1)
@@
 		(dnp no)
 		(property "Reference" "#FLG023"
-			(at 770.89 206.375 0)
+			(at 773.43 206.375 0)
 			(hide yes)
 			(show_name no)
@@
 		)
 		(property "Value" "PWR_FLAG"
-			(at 770.89 204.47 0)
+			(at 773.43 204.47 0)
+			(hide yes)
 			(show_name no)
 			(do_not_autoplace no)
@@
 		)
 		(property "Footprint" ""
-			(at 770.89 208.28 0)
+			(at 773.43 208.28 0)
 			(hide yes)
 			(show_name no)
@@
 		)
 		(property "Datasheet" "~"
-			(at 770.89 208.28 0)
+			(at 773.43 208.28 0)
 			(hide yes)
 			(show_name no)
@@
 		)
 		(property "Description" "Special symbol for telling ERC where power comes from"
-			(at 770.89 208.28 0)
+			(at 773.43 208.28 0)
 			(hide yes)
 			(show_name no)
@@
 	(symbol
 		(lib_id "Device:R_Small")
-		(at 768.35 208.28 270)
+		(at 758.19 208.28 270)
 		(unit 1)
 		(body_style 1)
@@
 		(dnp no)
 		(property "Reference" "R165"
-			(at 768.35 209.804 90)
+			(at 758.19 209.804 90)
 			(show_name no)
 			(do_not_autoplace no)
@@
 		)
 		(property "Value" "0.005"
-			(at 768.096 206.248 90)
+			(at 757.936 206.248 90)
 			(show_name no)
 			(do_not_autoplace no)
@@
 		)
 		(property "Footprint" "Resistor_SMD:R_2512_6332Metric"
-			(at 768.35 208.28 0)
+			(at 758.19 208.28 0)
 			(hide yes)
 			(show_name no)
@@
 		)
 		(property "Datasheet" ""
-			(at 768.35 208.28 0)
+			(at 758.19 208.28 0)
 			(hide yes)
 			(show_name no)
@@
 		)
 		(property "Description" "2W 5mΩ ±5% 2512 Current Sense Resistors - SMD/SMT ROHS"
-			(at 768.35 208.28 0)
+			(at 758.19 208.28 0)
 			(hide yes)
 			(show_name no)
@@
 		)
 		(property "Mfr. Part #" "FRM252WJR005TN"
-			(at 768.35 208.28 0)
+			(at 758.19 208.28 0)
 			(hide yes)
 			(show_name no)
@@
 		)
 		(property "LCSC Part #" "C7467241"
-			(at 768.35 208.28 0)
+			(at 758.19 208.28 0)
 			(hide yes)
 			(show_name no)
@@
 	(symbol
 		(lib_id "power:PWR_FLAG")
-		(at 755.65 208.28 0)
+		(at 740.41 205.74 0)
 		(unit 1)
 		(body_style 1)
@@
 		(fields_autoplaced yes)
 		(property "Reference" "#FLG012"
-			(at 755.65 206.375 0)
+			(at 740.41 203.835 0)
 			(hide yes)
 			(show_name no)
@@
 		)
 		(property "Value" "PWR_FLAG"
-			(at 755.65 203.2 0)
+			(at 740.41 200.66 0)
 			(hide yes)
 			(show_name no)
@@
 		)
 		(property "Footprint" ""
-			(at 755.65 208.28 0)
+			(at 740.41 205.74 0)
 			(hide yes)
 			(show_name no)
@@
 		)
 		(property "Datasheet" ""
-			(at 755.65 208.28 0)
+			(at 740.41 205.74 0)
 			(hide yes)
 			(show_name no)
@@
 		)
 		(property "Description" "Special symbol for telling ERC where power comes from"
-			(at 755.65 208.28 0)
+			(at 740.41 205.74 0)
 			(hide yes)
 			(show_name no)
