File: RASBB/Hardware/Rev.C/Design/RASBB.kicad_sch (KiCad schematic)
At the start: 71 parts, among them J20 Conn_01x02_Pin, SW1 435451019820, SW2 435451019820, U5 TLV9001DBVR

Commit message: RevC_06
Parts:
- C270: Manufacturer_Part_Number GRM155R71A104KA01D -> (none)
- C271: LCSC Part # (none) -> C1531; Manufacturer_Part_Number GRM1555C1H222JA01D -> (none); Mfr. Part # (none) -> 0402B222K500NT
- C272: Manufacturer_Part_Number GRM1555C1H222JA01D -> (none)
- J20: value Conn_01x02_Pin -> PWM_DAC_OUT
- R10, R9: value 4.7K -> 4K7; Mfr. Part #  WR04X4701FTL -> (none)
- R150: LCSC Part # (none) -> C95177; Manufacturer_Part_Number RC0603JR-070RL -> (none); Mfr. Part # (none) -> RC0603JR-070RL
- R151: LCSC Part # (none) -> C25804; Manufacturer_Part_Number RC0603FR-0710KL -> (none); Mfr. Part # (none) -> 0603WAF1002T5E
- R168, R169, R170, R171, R172, R173, R174, R175, R176, R177, R178, R179, R180, R181, R182, R183, R184: LCSC Part # C367410 -> C163808; Mfr. Part # WR02X1000FTL -> WR04X1000FTL
- R195, R200, R201: Manufacturer_Part_Number RC0603FR-0710KL -> (none)
- SW1, SW2: Part Number 435451019820 -> (none)
- U5: LCSC Part # (none) -> C19632595; Manufacturer_Part_Number TLV9001DBVR -> (none)
Connections:
- net 3V3 is gone; now on net Audio_IN-OUT/3V3: R10.2, R9.2
- net +3V3 renamed Audio_IN-OUT/3V3
- net Config-SPI FLASH/SCK_Flash_FPGA2 renamed Config-SPI FLASH/SCK_FLASH_FPGA2
- net Config-SPI FLASH/SI_Flash_FPGA2 renamed Config-SPI FLASH/SI_FLASH_FPGA2
- net Config-SPI FLASH/SO_Flash_FPGA2 renamed Config-SPI FLASH/SO_FLASH_FPGA2
Other:
- sheet Interconnect (page 11) renamed Interconnect
- sheet Audio_IN-OUT ports: added 3V3, 5V0; removed none
- sheet Config-SPI FLASH ports: added 3V3, CS_FLASH_FPGA2, CS_FLASH_uC, SCK_FLASH_FPGA2, SCK_FLASH_uC, SI_FLASH_FPGA2, SI_FLASH_uC, SO_FLASH_FPGA2, SO_FLASH_uC; removed CS_Flash_FPGA2, CS_Flash_uC, SCK_Flash_FPGA2, SCK_Flash_uC, SI_Flash_FPGA2, SI_Flash_uC, SO_Flash_FPGA2, SO_Flash_uC
- sheet Ethernet_FPGA ports: added 3V3; removed none
- sheet Ethernet_uC ports: added 3V3; removed none
- sheet FPGA-01 ports: added 1V0, 1V35, 1V8, 3V3; removed none
- sheet FPGA-02 ports: added 1V0, 1V35, 1V8, 3V3; removed none
- sheet HDMI ports: added 3V3, 5V0; removed none
- sheet Interconnect ports: added 3V3; removed none
- sheet PCIE ports: added 12V, 3V3, 5V0; removed none
- sheet POWER ports: added 12V, 1V0, 1V8, 5V0; removed none
- sheet RF_Transceiver ports: added 3V3; removed none
- sheet uController ports: added 3V3; removed none
- moved on the sheet: C270, C271, C272, J20, R1, R15, R150, R151, R16, R168, R169, R170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
