File: RASBB/Hardware/Rev.C/Design/RF_Transceiver.kicad_sch (KiCad schematic)
At the start: 21 parts, among them IC13 SX1280IMLTRT, J11 Conn_Coaxial, Y2 XC21M4-52.000-F10NNHPL

Commit message: RevC_06
Parts:
- C145, C149: Mfr. Part #  0402N200J500CT -> (none)
- C153: Mfr. Part # GRT155R71A474KE01D -> GRM155R71C474KE01D
- FB3: Mfr. Part #  BLM15BD601SH1D -> (none)
- J11: value Conn_Coaxial -> LORA_ANT
- L10: Mfr. Part #  FHW0402UC2N5KST -> (none)
- L9: Mfr. Part #  MHQ1005P3N0BT000 -> (none)
- Y2: Mfr. Part #  XC21M4-52.000-F10NNHPL -> (none)
Connections:
- net +3V3 renamed 3V3
Changed lines of the file:
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@@
 	(title_block
 		(title "RASBB")
-		(date "2026-09-20")
-		(rev "C")
+		(date "2026-09-27")
+		(rev "C.6")
 		(company "Mina Daneshpajouh")
 	)
@@
 			(width 0)
 			(type default)
+			(color 220 0 0 1)
 		)
 	)
@@
 			(width 0)
 			(type default)
+			(color 220 0 0 1)
 		)
 	)
@@
 		)
 	)
+	(hierarchical_label "3V3"
+		(shape input)
+		(at 22.86 124.46 90)
+		(effects
+			(font
+				(size 1.27 1.27)
+			)
+			(justify left)
+		)
+	)
 	(hierarchical_label "SPI_MOSI_LORA_G"
 		(shape input)
@@
 			)
 		)
-		(property "Mfr. Part # " "MHQ1005P3N0BT000"
-			(at 157.48 53.34 90)
-			(hide yes)
-			(show_name no)
-			(do_not_autoplace no)
-			(effects
-				(font
-					(size 1.27 1.27)
-				)
-			)
-		)
-		(property "LCSC Part # " ""
-			(at 157.48 53.34 90)
-			(hide yes)
-			(show_name no)
-			(do_not_autoplace no)
-			(effects
-				(font
-					(size 1.27 1.27)
-				)
-			)
-		)
 		(property "LCSC Part #" "C433005"
 			(at 157.48 53.34 0)
@@
 			)
 		)
-		(property "Mfr. Part #" "GRT155R71A474KE01D "
+		(property "Mfr. Part #" "GRM155R71C474KE01D"
 			(at 135.89 118.11 0)
 			(hide yes)
@@
 			)
 		)
-		(property "Mfr. Part # " "0402N200J500CT"
-			(at 78.74 57.15 0)
-			(hide yes)
-			(show_name no)
-			(do_not_autoplace no)
-			(effects
-				(font
-					(size 1.27 1.27)
-				)
-			)
-		)
 		(property "LCSC Part #" "C123468"
 			(at 78.74 57.15 0)
@@
 	)
 	(symbol
-		(lib_id "power:+3.3V")
-		(at 22.86 124.46 0)
-		(unit 1)
-		(body_style 1)
-		(exclude_from_sim no)
-		(in_bom yes)
-		(on_board yes)
-		(in_pos_files yes)
-		(dnp no)
-		(fields_autoplaced yes)
-		(property "Reference" "#PWR0137"
-			(at 22.86 128.27 0)
-			(hide yes)
-			(show_name no)
-			(do_not_autoplace no)
-			(effects
-				(font
-					(size 1.27 1.27)
-				)
-			)
-		)
-		(property "Value" "+3V3"
-			(at 25.4 123.1899 0)
-			(show_name no)
-			(do_not_autoplace no)
-			(effects
-				(font
-					(size 1.27 1.27)
-				)
-				(justify left)
-			)
-		)
-		(property "Footprint" ""
-			(at 22.86 124.46 0)
-			(hide yes)
-			(show_name no)
-			(do_not_autoplace no)
-			(effects
-				(font
-					(size 1.27 1.27)
-				)
-			)
-		)
-		(property "Datasheet" ""
-			(at 22.86 124.46 0)
-			(hide yes)
-			(show_name no)
-			(do_not_autoplace no)
-			(effects
-				(font
-					(size 1.27 1.27)
-				)
-			)
-		)
-		(property "Description" "Power symbol creates a global label with name \"+3.3V\""
-			(at 22.86 124.46 0)
-			(hide yes)
-			(show_name no)
-			(do_not_autoplace no)
-			(effects
-				(font
-					(size 1.27 1.27)
-				)
-			)
-		)
-		(pin "1"
-		)
-		(instances
-			(project "RASBB"
-				(path "/f6a5c334-5ee5-4dc9-84f1-7866383a3347/72084100-e3ab-4d46-b067-1f6f7a2f1c80"
-					(reference "#PWR0137")
-					(unit 1)
-				)
-			)
-		)
-	)
-	(symbol
 		(lib_id "Connector:Conn_Coaxial")
 		(at 228.6 53.34 0)
@@
 			)
 		)
-		(property "Value" "Conn_Coaxial"
+		(property "Value" "LORA_ANT"
 			(at 232.41 54.9031 0)
 			(show_name no)
@@
 			)
 		)
-		(property "Mfr. Part # " "XC21M4-52.000-F10NNHPL "
-			(at 68.58 69.85 0)
-			(hide yes)
-			(show_name no)
-			(do_not_autoplace no)
-			(effects
-				(font
-					(size 1.27 1.27)
-				)
-				(justify left)
-			)
-		)
 		(property "LCSC Part #" "C3034316"
 			(at 39.37 54.61 0)
@@
 			)
 		)
-		(property "Mfr. Part # " "BLM15BD601SH1D "
-			(at 41.91 113.03 0)
-			(hide yes)
-			(show_name no)
-			(do_not_autoplace no)
-			(effects
-				(font
-					(size 1.27 1.27)
-				)
-				(justify left)
-			)
-		)
-		(property "LCSC Part # " ""
-			(at 25.4 128.27 0)
-			(hide yes)
-			(show_name no)
-			(do_not_autoplace no)
-			(effects
-				(font
-					(size 1.27 1.27)
-				)
-			)
-		)
 		(property "LCSC Part #" "C710334"
 			(at 25.4 128.27 0)
@@
 			)
 		)
-		(property "Mfr. Part # " "FHW0402UC2N5KST"
-			(at 173.99 53.34 90)
-			(hide yes)
-			(show_name no)
-			(do_not_autoplace no)
-			(effects
-				(font
-					(size 1.27 1.27)
-				)
-			)
-		)
-		(property "LCSC Part # " ""
-			(at 173.99 53.34 90)
-			(hide yes)
-			(show_name no)
-			(do_not_autoplace no)
-			(effects
-				(font
-					(size 1.27 1.27)
-				)
-			)
-		)
 		(property "LCSC Part #" "C317668"
 			(at 173.99 53.34 0)
@@
 			(at 36.83 60.96 0)
 			(hide yes)
-			(show_name no)
-			(do_not_autoplace no)
-			(effects
-				(font
-					(size 1.27 1.27)
-				)
-			)
-		)
-		(property "Mfr. Part # " "0402N200J500CT"
-			(at 36.83 60.96 0)
-			(hide yes)
