File: RASBB/Hardware/Rev.C/Design/uController.kicad_sch (KiCad schematic)
At the start: 68 parts, among them IC12 STM32H743VGT6, J10 ZX-PZ1.27-2-5PWZ, J7 USB_C_Receptacle, J8 ZX-PZ1.27-2-5PWZ, J9 KF2EDGR-3.5-2P, Q1 DMN6075S, U6 CH340E, U7 AHT20, Y1 X503220MSB2GI

Commit message: RevC_06
Parts:
- C139, C140: Mfr. Part #  0402N200J500CT -> (none)
- D27: footprint DIOM5026X229N -> RASBB:DIOM5026X229N; Manufacturer_Part_Number SMAJ33A -> (none)
- D6: Mfr. Part #   S210_R1_00001 -> (none)
- D7: LCSC Part #   C5355433 -> (none); Mfr. Part #   A-SP192YR6C-C01-4T -> (none)
- D8: LCSC Part #   C19171301 -> (none); Mfr. Part #   A-SP192DGHC-C01-4T -> (none)
- D9: LCSC Part #   C5355434 -> (none); Mfr. Part #   A-SP192GS1D-C01-4T -> (none)
- FB1, FB2: Mfr. Part #  BLM15BD601SH1D -> (none)
- IC12: Mfr. Part #  STM32H743VGT6 -> (none)
- J10: value ZX-PZ1.27-2-5PWZ -> STM32_JTAG; Mfr. Part #  ZX-PZ1.27-2-5PWZ -> (none)
- J7: value USB_C_Receptacle -> USB_UART; LCSC Part #   C2765186 -> (none); Mfr. Part #   TYPE-C 16PIN 2MD(073) -> (none)
- J8: value ZX-PZ1.27-2-5PWZ -> STM32_DEBUG; Mfr. Part #  ZX-PZ1.27-2-5PWZ -> (none)
- J9: value KF2EDGR-3.5-2P -> ALARM_OUT; LCSC Part #   C441171 -> (none); Mfr. Part #   KF2EDGR-3.5-2P -> (none)
- Q1: LCSC Part #   C5122015 -> (none); Mfr. Part #   DMN6075S -> (none)
- R101, R114, R115, R116, R117, R118, R119, R120: value 4.7K -> 4K7; Mfr. Part #  WR04X4701FTL -> (none)
- R102: Mfr. Part #   MR04X000PTL -> (none)
- R97, R98: Mfr. Part #   WR04X512JTL -> (none)
- S1: LCSC Part #   C87038 -> (none); Mfr. Part #   B3FS-1002P -> (none)
- U6: LCSC Part #   C99652 -> (none); Mfr. Part #   CH340E -> (none)
- U7: Mfr. Part #  AHT20 -> (none)
- Y1: Mfr. Part #  X503220MSB2GI -> (none)
Connections:
- net +3V3 renamed 3V3
